File: peripherals/glucometer-pcb.kicad_sch (KiCad schematic)
At the start: 17 parts, among them IC1 RC4558IP, IC2 LM1458N, IC3 RC4558IP

Commit message: change name
Parts:
- removed TP3: (no value), TestPoint:TestPoint_Keystone_5015_Micro-Minature, symbol Connector:TestPoint
- added BZ1: Buzzer, Buzzer_Beeper:MagneticBuzzer_Kingstate_KCG0601, symbol Device:Buzzer
- added D1: LED, LED_THT:LED_D3.0mm_Clear, symbol Device:LED
- added D2: LED, LED_THT:LED_D3.0mm_FlatTop, symbol Device:LED
- added R3: 120, Resistor_THT:R_Axial_DIN0204_L3.6mm_D1.6mm_P7.62mm_Horizontal, symbol Device:R
- added R4: 240, Resistor_THT:R_Axial_DIN0204_L3.6mm_D1.6mm_P7.62mm_Horizontal, symbol Device:R
- added U1: ESP32_DevKit_V1_DOIT, esp32_devkit_v1_doit:esp32_devkit_v1_doit, symbol esp32_devkit_v1_doit:ESP32_DevKit_V1_DOIT
- renumbered D1 to D3, R3 to R5, R4 to R6, R5 to R7, R6 to R8, R7 to R9
Connections:
- net VCC: now also D1.1 (K), U1.1 (3V3)
- net SIGNAL_OUT: now reaches IC3.6 (2IN-), R8.1, R9.2
- net SIGNAL_OUT: now also U1.8 (D5)
- new net: D2.1 (K), R4.2, U1.17 (GND)
- new net: D2.2 (A), U1.23 (D25)
- new net: BZ1.2 (+), R3.1
- new net: R3.2, U1.2 (GND)
- new net: D1.2 (A), R4.1
- new net: BZ1.1 (-), U1.4 (D2)

Commit message: emmiter circuit
Parts:
- removed C1: 10u, Capacitor_THT:CP_Radial_Tantal_D7.0mm_P5.00mm, symbol Device:C
- removed C2: 15p, Capacitor_THT:CP_Radial_D8.0mm_P3.80mm, symbol Device:C
- removed C3: 100n, Capacitor_THT:CP_Radial_Tantal_D7.0mm_P5.00mm, symbol Device:C
- removed D3: D_Photo, LED_SMD:LED_2010_5025Metric, symbol Device:D_Photo
- removed IC1, IC3: RC4558IP, Custom:DIP794W53P254L959H508Q8N, symbol RC4558IP:RC4558IP
- removed IC2: LM1458N, Custom:MC1458N, symbol LM1458N:LM1458N
- removed R1, R2: 10k, Resistor_THT:R_Axial_DIN0204_L3.6mm_D1.6mm_P7.62mm_Horizontal, symbol Device:R
- removed R5: 25k, Resistor_THT:R_Axial_DIN0204_L3.6mm_D1.6mm_P7.62mm_Horizontal, symbol Device:R
- removed R6, R9: 100k, Resistor_THT:R_Axial_DIN0204_L3.6mm_D1.6mm_P7.62mm_Horizontal, symbol Device:R
- removed R7: 330k, Resistor_THT:R_Axial_DIN0204_L3.6mm_D1.6mm_P7.62mm_Horizontal, symbol Device:R
- removed R8: 1k, Resistor_THT:R_Axial_DIN0204_L3.6mm_D1.6mm_P7.62mm_Horizontal, symbol Device:R
- removed TP2: TestPoint, TestPoint:TestPoint_Keystone_5015_Micro-Minature, symbol Connector:TestPoint
- added 3V3_OUT1: TestPoint, TestPoint:TestPoint_Keystone_5015_Micro-Minature, symbol Connector:TestPoint
- added BT1: Battery_Cell, Connector_Wire:SolderWire-0.1sqmm_1x02_P3.6mm_D0.4mm_OD1mm, symbol Device:Battery_Cell
- added R3: 120, Resistor_THT:R_Axial_DIN0204_L3.6mm_D1.6mm_P7.62mm_Horizontal, symbol Device:R
- D2: renamed from D1; value LED -> EMITTER
- R2: renamed from R4; value 240 -> 120
- U1: value ESP32_DevKit_V1_DOIT -> (none); footprint esp32_devkit_v1_doit:esp32_devkit_v1_doit -> (none)
- renumbered D2 to D1, R3 to R1
Connections:
- net GND: now also R1.2, R2.2, U1.14 (GND), U1.17 (GND), BT1.2 (-), R3.2; no longer TP1.1
- net SIGNAL_OUT: now also TP1.1
- net VCC: now also U1.16 (3V3), 3V3_OUT1.1; no longer D2.1 (K), U1.1 (3V3)
- net at D1.2 (A): now also U1.11 (IO14); no longer U1.23 (D25)
- net at U1.2 (SENSOR_VP): no longer R1.2
- net at R2.1: now also D1.1 (K); no longer D2.2 (A)
- net at BZ1.1 (-): now also U1.19 (IO2); no longer U1.4 (D2)
- net at U1.15 (VIN): now also BT1.1 (+)
- net at U1.18 (IO15): now also D2.2 (A)
- new net: D2.1 (K), R3.1
- no-connect marks 6 -> 22
Other:
- moved on the sheet: BZ1, D1, D2, R1, R2

Commit message: fixed PCB
Parts:
- U1: value (none) -> ESP32_DevKit_V1_DOIT; footprint (none) -> esp32_devkit_v1_doit:esp32_devkit_v1_doit
Connections:
- net INTERRUPT_PIN_BTN: now reaches U1.30 (IO23)
- no-connect marks 22 -> 21
Changed lines of the file:
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@@
   (no_connect (at 83.82 119.38))
   (no_connect (at 83.82 106.68))
-  (no_connect (at 83.82 101.6))
   (no_connect (at 83.82 99.06))
   (no_connect (at 83.82 96.52))
@@
     (stroke (width 0) (type default) (color 0 0 0 0))
   )
+  (wire (pts (xy 83.82 101.6) (xy 109.22 101.6))
+    (stroke (width 0) (type default) (color 0 0 0 0))
+  )
   (wire (pts (xy 68.58 34.29) (xy 68.58 39.37))
     (stroke (width 0) (type default) (color 0 0 0 0))
@@
     (stroke (width 0) (type default) (color 0 0 0 0))
   )
+  (wire (pts (xy 109.22 97.79) (xy 109.22 101.6))
+    (stroke (width 0) (type default) (color 0 0 0 0))
+  )
   (wire (pts (xy 87.63 66.04) (xy 83.82 66.04))
     (stroke (width 0) (type default) (color 0 0 0 0))
   )
   (wire (pts (xy 96.52 111.76) (xy 92.71 111.76))
+    (stroke (width 0) (type default) (color 0 0 0 0))
+  )
+  (wire (pts (xy 109.22 97.79) (xy 110.49 97.79))
     (stroke (width 0) (type default) (color 0 0 0 0))
   )
@@
     (property "Referencias entre hojas" "${INTERSHEET_REFS}" (id 0) (at 90.2364 65.9606 0)
       (effects (font (size 1.27 1.27)) (justify right) hide)
+    )
+  )
+  (global_label "INTERRUPT_PIN_BTN" (shape input) (at 110.49 97.79 0) (fields_autoplaced)
+    (effects (font (size 1.27 1.27)) (justify left))
+    (property "Referencias entre hojas" "${INTERSHEET_REFS}" (id 0) (at 131.7717 97.7106 0)
+      (effects (font (size 1.27 1.27)) (justify left) hide)
     )
   )
@@
       (effects (font (size 1.27 1.27)) (justify left))
     )
-    (property "Value" "" (id 1) (at 70.5994 55.88 0)
-      (effects (font (size 1.27 1.27)) (justify left))
-    )
-    (property "Footprint" "" (id 2) (at 57.15 57.15 0)
-      (effects (font (size 1.27 1.27)) hide)
-    )
+    (property "Value" "ESP32_DevKit_V1_DOIT" (id 1) (at 70.5994 55.88 0)
+      (effects (font (size 1.27 1.27)) (justify left))
+    )
+    (property "Footprint" "esp32_devkit_v1_doit:esp32_devkit_v1_doit" (id 2) (at 57.15 57.15 0)
+      (effects (font (size 1.27 1.27)) hide)
+    )

Commit message: fixed PCB
Parts:
- added INTERRUPT_GPIO18: SW_Push, symbol Switch:SW_Push
- added OLED_PINS: (no value), symbol Connector:Conn_01x04_Female
- renumbered BT1 to BATTERY1, R2 to R1, R3 to R2, R1 to R3, TP1 to SIGNAL_IN1, D1 to Testigo1
Connections:
- net INTERRUPT_PIN_BTN is gone; now on an unnamed net: U1.30 (IO23)
- net GND: now also INTERRUPT_GPIO18.2, OLED_PINS.1 (Pin_1)
- net VCC: now also OLED_PINS.2 (Pin_2)
- net at Testigo1.2 (A): now also U1.29 (IO22); no longer U1.11 (IO14)
- net at D2.2 (A): no longer U1.18 (IO15)
- net at BZ1.1 (-): now also U1.24 (IO18); no longer U1.19 (IO2)
- net at U1.21 (IO16): now also OLED_PINS.3 (Pin_3)
- net at U1.22 (IO17): now also OLED_PINS.4 (Pin_4)
- net at U1.25 (IO19): now also INTERRUPT_GPIO18.1
- net at U1.26 (IO21): now also SIGNAL_IN1.1
- net SIGNAL_OUT: no longer names the net of U1.8 (IO25)
- net SIGNAL_OUT: no longer SIGNAL_IN1.1
- no-connect marks 21 -> 19
Other:
- moved on the sheet: BZ1, D2, R1, R2, R3, SIGNAL_IN1, Testigo1

Commit message: changes
Parts:
- INTERRUPT_GPIO1: renamed from INTERRUPT_GPIO18; footprint (none) -> Connector_Wire:SolderWire-0.1sqmm_1x02_P3.6mm_D0.4mm_OD1mm
- OLED_PINS1: renamed from OLED_PINS; value (none) -> Conn_01x04_Female; footprint (none) -> Connector_Wire:SolderWire-0.1sqmm_1x04_P3.6mm_D0.4mm_OD1mm
- renumbered D2 to D1, R3 to R1, R1 to R2, R2 to R3
Connections:
- net at Testigo1.2 (A): now also U1.8 (IO25); no longer U1.29 (IO22)
- net at OLED_PINS1.3 (Pin_3): now also U1.26 (IO21); no longer U1.21 (IO16)
- net at OLED_PINS1.4 (Pin_4): now also U1.29 (IO22); no longer U1.22 (IO17)
- net at SIGNAL_IN1.1: now also U1.21 (IO16); no longer U1.26 (IO21)
Other:
- moved on the sheet: D1, OLED_PINS1, R2, R3, SIGNAL_IN1, Testigo1

Commit message: last update emmiter pcb
Parts:
- removed R2: 120, Resistor_THT:R_Axial_DIN0204_L3.6mm_D1.6mm_P7.62mm_Horizontal, symbol Device:R
- removed Testigo1: LED, LED_THT:LED_D3.0mm_FlatTop, symbol Device:LED
Connections:
- net at SIGNAL_IN1.1: now also U1.9 (IO26); no longer U1.21 (IO16)
- net VCC: no longer names the net of 3V3_OUT1.1, OLED_PINS1.2 (Pin_2), U1.16 (3V3)
- no-connect marks 19 -> 20
Other:
- moved on the sheet: SIGNAL_IN1
Changed lines of the file:
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@@
 (kicad_sch (version 20211123) (generator eeschema)
   (paper "A4")
-  (junction (at 68.58 39.37) (diameter 0) (color 0 0 0 0)
-  )
   (junction (at 68.58 48.26) (diameter 0) (color 0 0 0 0)
   )
@@
   (no_connect (at 83.82 63.5))
   (no_connect (at 83.82 109.22))
-  (no_connect (at 83.82 114.3))
   (no_connect (at 83.82 116.84))
   (no_connect (at 83.82 111.76))
@@
   (no_connect (at 83.82 83.82))
   (no_connect (at 83.82 66.04))
-  (no_connect (at 83.82 106.68))
-  (wire (pts (xy 83.82 104.14) (xy 106.68 104.14))
-    (stroke (width 0) (type default) (color 0 0 0 0))
-  )
-  (wire (pts (xy 87.63 86.36) (xy 87.63 76.2))
+  (no_connect (at 83.82 104.14))
+  (no_connect (at 83.82 114.3))
+  (no_connect (at 83.82 86.36))
+  (wire (pts (xy 83.82 106.68) (xy 97.79 106.68))
     (stroke (width 0) (type default) (color 0 0 0 0))
   )
@@
     (stroke (width 0) (type default) (color 0 0 0 0))
   )
-  (wire (pts (xy 68.58 127) (xy 68.58 133.35))
-    (stroke (width 0) (type default) (color 0 0 0 0))
-  )
   (wire (pts (xy 83.82 99.06) (xy 171.45 99.06))
     (stroke (width 0) (type default) (color 0 0 0 0))
@@
     (stroke (width 0) (type default) (color 0 0 0 0))
   )
-  (wire (pts (xy 66.04 127) (xy 66.04 133.35))
-    (stroke (width 0) (type default) (color 0 0 0 0))
-  )
   (wire (pts (xy 154.94 93.98) (xy 154.94 48.26))
     (stroke (width 0) (type default) (color 0 0 0 0))
@@
     (stroke (width 0) (type default) (color 0 0 0 0))
   )
-  (wire (pts (xy 83.82 86.36) (xy 87.63 86.36))
-    (stroke (width 0) (type default) (color 0 0 0 0))
-  )
   (wire (pts (xy 66.04 48.26) (xy 66.04 55.88))
     (stroke (width 0) (type default) (color 0 0 0 0))
   )
-  (wire (pts (xy 68.58 34.29) (xy 68.58 39.37))
-    (stroke (width 0) (type default) (color 0 0 0 0))
-  )
   (wire (pts (xy 83.82 91.44) (xy 111.76 91.44))
     (stroke (width 0) (type default) (color 0 0 0 0))
   )
-  (wire (pts (xy 128.27 104.14) (xy 124.46 104.14))
-    (stroke (width 0) (type default) (color 0 0 0 0))
-  )
   (wire (pts (xy 83.82 96.52) (xy 171.45 96.52))
     (stroke (width 0) (type default) (color 0 0 0 0))
@@
     (stroke (width 0) (type default) (color 0 0 0 0))
   )
+  (wire (pts (xy 66.04 127) (xy 66.04 129.54))
+    (stroke (width 0) (type default) (color 0 0 0 0))
+  )
   (wire (pts (xy 109.22 86.36) (xy 111.76 86.36))
     (stroke (width 0) (type default) (color 0 0 0 0))
@@
     (stroke (width 0) (type default) (color 0 0 0 0))
   )
-  (wire (pts (xy 87.63 76.2) (xy 88.9 76.2))
-    (stroke (width 0) (type default) (color 0 0 0 0))
-  )
   (wire (pts (xy 134.62 93.98) (xy 135.89 93.98))
     (stroke (width 0) (type default) (color 0 0 0 0))
@@
     (stroke (width 0) (type default) (color 0 0 0 0))
   )
-  (wire (pts (xy 116.84 104.14) (xy 114.3 104.14))
+  (wire (pts (xy 68.58 127) (xy 68.58 129.54))
     (stroke (width 0) (type default) (color 0 0 0 0))
   )
@@
     )
   )
+  (global_label "GND" (shape input) (at 68.58 129.54 0) (fields_autoplaced)
+    (effects (font (size 1.27 1.27)) (justify left))
+    (property "Referencias entre hojas" "${INTERSHEET_REFS}" (id 0) (at 74.8636 129.4606 0)
+      (effects (font (size 1.27 1.27)) (justify left) hide)
+    )
+  )
   (global_label "GND" (shape input) (at 100.33 86.36 180) (fields_autoplaced)
     (effects (font (size 1.27 1.27)) (justify right))
@@
     )
   )
-  (global_label "GND" (shape input) (at 68.58 133.35 0) (fields_autoplaced)
-    (effects (font (size 1.27 1.27)) (justify left))
-    (property "Referencias entre hojas" "${INTERSHEET_REFS}" (id 0) (at 74.8636 133.4294 0)
-      (effects (font (size 1.27 1.27)) (justify left) hide)
-    )
-  )
-  (global_label "GND" (shape input) (at 128.27 104.14 270) (fields_autoplaced)
+  (global_label "GND" (shape input) (at 66.04 129.54 180) (fields_autoplaced)
     (effects (font (size 1.27 1.27)) (justify right))
-    (property "Referencias entre hojas" "${INTERSHEET_REFS}" (id 0) (at 128.1906 110.4236 90)
+    (property "Referencias entre hojas" "${INTERSHEET_REFS}" (id 0) (at 59.7564 129.4606 0)
       (effects (font (size 1.27 1.27)) (justify right) hide)
     )
@@
     )
   )
-  (global_label "GND" (shape input) (at 66.04 133.35 180) (fields_autoplaced)
-    (effects (font (size 1.27 1.27)) (justify right))
-    (property "Referencias entre hojas" "${INTERSHEET_REFS}" (id 0) (at 59.7564 133.2706 0)
-      (effects (font (size 1.27 1.27)) (justify right) hide)
-    )
-  )
-  (global_label "VCC" (shape input) (at 68.58 34.29 90) (fields_autoplaced)
-    (effects (font (size 1.27 1.27)) (justify left))
-    (property "Referencias entre hojas" "${INTERSHEET_REFS}" (id 0) (at 68.5006 28.2483 90)
-      (effects (font (size 1.27 1.27)) (justify left) hide)
-    )
-  )
   (global_label "GND" (shape input) (at 135.89 93.98 0) (fields_autoplaced)
     (effects (font (size 1.27 1.27)) (justify left))
-    (property "Referencias entre hojas" "${INTERSHEET_REFS}" (id 0) (at 142.1736 94.0594 0)
+    (property "Referencias entre hojas" "${INTERSHEET_REFS}" (id 0) (at 142.1736 93.9006 0)
       (effects (font (size 1.27 1.27)) (justify left) hide)
     )
-  )
-  (symbol (lib_id "Device:LED") (at 110.49 104.14 180) (unit 1)
-    (in_bom yes) (on_board yes)
-    (property "Reference" "Testigo1" (id 0) (at 113.3476 106.68 90)
-      (effects (font (size 1.27 1.27)) (justify left))
-    )
-    (property "Value" "LED" (id 1) (at 110.8076 106.68 90)
-      (effects (font (size 1.27 1.27)) (justify left))
-    )
-    (property "Footprint" "LED_THT:LED_D3.0mm_FlatTop" (id 2) (at 110.49 104.14 0)
-      (effects (font (size 1.27 1.27)) hide)
-    )
-    (property "Datasheet" "~" (id 3) (at 110.49 104.14 0)
-      (effects (font (size 1.27 1.27)) hide)
-    )
-    (pin "1")
-    (pin "2")
   )
   (symbol (lib_id "Connector:Conn_01x04_Female") (at 176.53 93.98 0) (unit 1)
@@
     (pin "2")
   )
-  (symbol (lib_id "Connector:TestPoint") (at 88.9 76.2 0) (mirror y) (unit 1)
-    (in_bom yes) (on_board yes) (fields_autoplaced)
-    (property "Reference" "SIGNAL_IN1" (id 0) (at 91.44 71.6279 0)
+  (symbol (lib_id "Connector:TestPoint") (at 97.79 106.68 270) (mirror x) (unit 1)
+    (in_bom yes) (on_board yes) (fields_autoplaced)
+    (property "Reference" "SIGNAL_IN1" (id 0) (at 102.3621 109.22 0)
       (effects (font (size 1.27 1.27)) (justify right))
     )
-    (property "Value" "TestPoint" (id 1) (at 91.44 74.1679 0)
+    (property "Value" "TestPoint" (id 1) (at 99.8221 109.22 0)
       (effects (font (size 1.27 1.27)) (justify right))
     )
-    (property "Footprint" "TestPoint:TestPoint_Keystone_5015_Micro-Minature" (id 2) (at 83.82 76.2 0)
-      (effects (font (size 1.27 1.27)) hide)
-    )
-    (property "Datasheet" "~" (id 3) (at 83.82 76.2 0)
+    (property "Footprint" "TestPoint:TestPoint_Keystone_5015_Micro-Minature" (id 2) (at 97.79 101.6 0)
+      (effects (font (size 1.27 1.27)) hide)
+    )
+    (property "Datasheet" "~" (id 3) (at 97.79 101.6 0)
       (effects (font (size 1.27 1.27)) hide)
     )
@@
     )
     (property "Datasheet" "~" (id 3) (at 129.54 88.9 0)
-      (effects (font (size 1.27 1.27)) hide)
-    )
-    (pin "1")
-    (pin "2")
-  )
-  (symbol (lib_id "Device:R") (at 120.65 104.14 90) (unit 1)
-    (in_bom yes) (on_board yes) (fields_autoplaced)
-    (property "Reference" "R2" (id 0) (at 121.9201 106.68 0)
-      (effects (font (size 1.27 1.27)) (justify right))
-    )
-    (property "Value" "120" (id 1) (at 119.3801 106.68 0)
-      (effects (font (size 1.27 1.27)) (justify right))
-    )
-    (property "Footprint" "Resistor_THT:R_Axial_DIN0204_L3.6mm_D1.6mm_P7.62mm_Horizontal" (id 2) (at 120.65 105.918 90)
-      (effects (font (size 1.27 1.27)) hide)
-    )
-    (property "Datasheet" "~" (id 3) (at 120.65 104.14 0)
       (effects (font (size 1.27 1.27)) hide)
     )
@@
       (reference "R1") (unit 1) (value "120") (footprint "Resistor_THT:R_Axial_DIN0204_L3.6mm_D1.6mm_P7.62mm_Horizontal")
     )
-    (path "/b6a30bc2-0d74-43ed-aa2b-a3d443bd9193"
-      (reference "R2") (unit 1) (value "120") (footprint "Resistor_THT:R_Axial_DIN0204_L3.6mm_D1.6mm_P7.62mm_Horizontal")
-    )
     (path "/48716155-f70c-423a-8030-4a2d322cc6d9"
       (reference "R3") (unit 1) (value "120") (footprint "Resistor_THT:R_Axial_DIN0204_L3.6mm_D1.6mm_P7.62mm_Horizontal")
@@
       (reference "SIGNAL_IN1") (unit 1) (value "TestPoint") (footprint "TestPoint:TestPoint_Keystone_5015_Micro-Minature")
     )
-    (path "/019be3e5-53d3-4756-bc1c-bd7873df24c4"
-      (reference "Testigo1") (unit 1) (value "LED") (footprint "LED_THT:LED_D3.0mm_FlatTop")
-    )
     (path "/d6ca7d44-4b9c-4d66-afa6-a65a2e89d1cd"

Commit message: last update
Connections:
- net at SIGNAL_IN1.1: now also U1.4 (IO34); no longer U1.9 (IO26)
Other:
- moved on the sheet: SIGNAL_IN1
Changed lines of the file:
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@@
   (junction (at 68.58 48.26) (diameter 0) (color 0 0 0 0)
   )
+  (no_connect (at 83.82 106.68))
   (no_connect (at 83.82 81.28))
+  (no_connect (at 83.82 71.12))
+  (no_connect (at 83.82 78.74))
   (no_connect (at 53.34 66.04))
   (no_connect (at 53.34 68.58))
   (no_connect (at 53.34 60.96))
-  (no_connect (at 83.82 78.74))
   (no_connect (at 83.82 76.2))
   (no_connect (at 83.82 73.66))
-  (no_connect (at 83.82 71.12))
   (no_connect (at 83.82 68.58))
   (no_connect (at 83.82 63.5))
   (no_connect (at 83.82 109.22))
-  (no_connect (at 83.82 116.84))
   (no_connect (at 83.82 111.76))
   (no_connect (at 83.82 119.38))
@@
   (no_connect (at 83.82 114.3))
   (no_connect (at 83.82 86.36))
-  (wire (pts (xy 83.82 106.68) (xy 97.79 106.68))
-    (stroke (width 0) (type default) (color 0 0 0 0))
-  )
   (wire (pts (xy 83.82 101.6) (xy 189.23 101.6))
     (stroke (width 0) (type default) (color 0 0 0 0))
@@
   )
   (wire (pts (xy 68.58 48.26) (xy 68.58 55.88))
+    (stroke (width 0) (type default) (color 0 0 0 0))
+  )
+  (wire (pts (xy 83.82 116.84) (xy 97.79 116.84))
     (stroke (width 0) (type default) (color 0 0 0 0))
   )
@@
   )
   (symbol (lib_id "Device:R") (at 105.41 86.36 270) (mirror x) (unit 1)
-    (in_bom yes) (on_board yes) (fields_autoplaced)
-    (property "Reference" "R1" (id 0) (at 105.41 80.01 90))
+    (in_bom yes) (on_board yes)
+    (property "Reference" "R1" (id 0) (at 87.63 129.54 0))
     (property "Value" "120" (id 1) (at 105.41 82.55 90))
     (property "Footprint" "Resistor_THT:R_Axial_DIN0204_L3.6mm_D1.6mm_P7.62mm_Horizontal" (id 2) (at 105.41 88.138 90)
@@
     (pin "2")
   )
-  (symbol (lib_id "Connector:TestPoint") (at 97.79 106.68 270) (mirror x) (unit 1)
-    (in_bom yes) (on_board yes) (fields_autoplaced)
-    (property "Reference" "SIGNAL_IN1" (id 0) (at 102.3621 109.22 0)
-      (effects (font (size 1.27 1.27)) (justify right))
-    )
-    (property "Value" "TestPoint" (id 1) (at 99.8221 109.22 0)
-      (effects (font (size 1.27 1.27)) (justify right))
-    )
-    (property "Footprint" "TestPoint:TestPoint_Keystone_5015_Micro-Minature" (id 2) (at 97.79 101.6 0)
-      (effects (font (size 1.27 1.27)) hide)
-    )
-    (property "Datasheet" "~" (id 3) (at 97.79 101.6 0)
-      (effects (font (size 1.27 1.27)) hide)
-    )
+  (symbol (lib_id "Connector:TestPoint") (at 97.79 116.84 270) (mirror x) (unit 1)
+    (in_bom yes) (on_board yes) (fields_autoplaced)
+    (property "Reference" "SIGNAL_IN1" (id 0) (at 102.3621 119.38 0)
+      (effects (font (size 1.27 1.27)) (justify right))
+    )
+    (property "Value" "TestPoint" (id 1) (at 99.8221 119.38 0)
+      (effects (font (size 1.27 1.27)) (justify right))
+    )
+    (property "Footprint" "TestPoint:TestPoint_Keystone_5015_Micro-Minature" (id 2) (at 97.79 111.76 0)
+      (effects (font (size 1.27 1.27)) hide)
+    )
+    (property "Datasheet" "~" (id 3) (at 97.79 111.76 0)
+      (effects (font (size 1.27 1.27)) hide)
+    )
