File: peripherals/glucometer-pcb.kicad_pcb (KiCad board)
At the start: 2 copper layers, 54.8 x 66.9 mm, 15 parts, among them U1 ESP32_DevKit_V1_DOIT

Commit message: added prints
Parts:
- added 100nF2: CAP, Capacitor_THT:C_Disc_D4.3mm_W1.9mm_P5.00mm, B.Cu at (120.0, 67.1)
- added 100nF3: CAP, Capacitor_THT:C_Disc_D4.3mm_W1.9mm_P5.00mm, B.Cu at (185.0, 67.1)
- added 100nF4: CAP, Capacitor_THT:C_Disc_D4.3mm_W1.9mm_P5.00mm, B.Cu at (250.0, 67.1)
- added 100nF5: CAP, Capacitor_THT:C_Disc_D4.3mm_W1.9mm_P5.00mm, B.Cu at (55.0, 147.1)
- added 100nF6: CAP, Capacitor_THT:C_Disc_D4.3mm_W1.9mm_P5.00mm, B.Cu at (120.0, 147.1)
- added 100nF7: CAP, Capacitor_THT:C_Disc_D4.3mm_W1.9mm_P5.00mm, B.Cu at (185.0, 147.1)
- added 100nF8: CAP, Capacitor_THT:C_Disc_D4.3mm_W1.9mm_P5.00mm, B.Cu at (250.0, 147.1)
- added 3V3_OUT2: TestPoint, TestPoint:TestPoint_Keystone_5015_Micro-Minature, B.Cu at (108.6, 19.2)
- added 3V3_OUT3: TestPoint, TestPoint:TestPoint_Keystone_5015_Micro-Minature, B.Cu at (173.6, 19.2)
- added 3V3_OUT4: TestPoint, TestPoint:TestPoint_Keystone_5015_Micro-Minature, B.Cu at (238.6, 19.2)
- added 3V3_OUT5: TestPoint, TestPoint:TestPoint_Keystone_5015_Micro-Minature, B.Cu at (43.6, 99.2)
- added 3V3_OUT6: TestPoint, TestPoint:TestPoint_Keystone_5015_Micro-Minature, B.Cu at (108.6, 99.2)
- added 3V3_OUT7: TestPoint, TestPoint:TestPoint_Keystone_5015_Micro-Minature, B.Cu at (173.6, 99.2)
- added 3V3_OUT8: TestPoint, TestPoint:TestPoint_Keystone_5015_Micro-Minature, B.Cu at (238.6, 99.2)
- added BATTERY2: Battery_Cell, Connector_Wire:SolderWire-0.1sqmm_1x02_P3.6mm_D0.4mm_OD1mm, B.Cu at (127.5, 19.4)
- added BATTERY3: Battery_Cell, Connector_Wire:SolderWire-0.1sqmm_1x02_P3.6mm_D0.4mm_OD1mm, B.Cu at (192.5, 19.4)
- added BATTERY4: Battery_Cell, Connector_Wire:SolderWire-0.1sqmm_1x02_P3.6mm_D0.4mm_OD1mm, B.Cu at (257.5, 19.4)
- added BATTERY5: Battery_Cell, Connector_Wire:SolderWire-0.1sqmm_1x02_P3.6mm_D0.4mm_OD1mm, B.Cu at (62.5, 99.4)
- added BATTERY6: Battery_Cell, Connector_Wire:SolderWire-0.1sqmm_1x02_P3.6mm_D0.4mm_OD1mm, B.Cu at (127.5, 99.4)
- added BATTERY7: Battery_Cell, Connector_Wire:SolderWire-0.1sqmm_1x02_P3.6mm_D0.4mm_OD1mm, B.Cu at (192.5, 99.4)
- added BATTERY8: Battery_Cell, Connector_Wire:SolderWire-0.1sqmm_1x02_P3.6mm_D0.4mm_OD1mm, B.Cu at (257.5, 99.4)
- added BZ2: Buzzer, Buzzer_Beeper:MagneticBuzzer_ProSignal_ABI-009-RC, B.Cu at (95.1, 44.7)
- added BZ3: Buzzer, Buzzer_Beeper:MagneticBuzzer_ProSignal_ABI-009-RC, B.Cu at (160.1, 44.7)
- added BZ4: Buzzer, Buzzer_Beeper:MagneticBuzzer_ProSignal_ABI-009-RC, B.Cu at (225.1, 44.7)
- added BZ5: Buzzer, Buzzer_Beeper:MagneticBuzzer_ProSignal_ABI-009-RC, B.Cu at (30.1, 124.7)
- added BZ6: Buzzer, Buzzer_Beeper:MagneticBuzzer_ProSignal_ABI-009-RC, B.Cu at (95.1, 124.7)
- added BZ7: Buzzer, Buzzer_Beeper:MagneticBuzzer_ProSignal_ABI-009-RC, B.Cu at (160.1, 124.7)
- added BZ8: Buzzer, Buzzer_Beeper:MagneticBuzzer_ProSignal_ABI-009-RC, B.Cu at (225.1, 124.7)
- added D2: EMITTER, LED_THT:LED_D3.0mm_Clear, F.Cu at (117.6, 80.6)
- added D3: EMITTER, LED_THT:LED_D3.0mm_Clear, F.Cu at (182.6, 80.6)
- added D4: EMITTER, LED_THT:LED_D3.0mm_Clear, F.Cu at (247.6, 80.6)
- added D5: EMITTER, LED_THT:LED_D3.0mm_Clear, F.Cu at (52.6, 160.6)
- added D6: EMITTER, LED_THT:LED_D3.0mm_Clear, F.Cu at (117.6, 160.6)
- added D7: EMITTER, LED_THT:LED_D3.0mm_Clear, F.Cu at (182.6, 160.6)
- added D8: EMITTER, LED_THT:LED_D3.0mm_Clear, F.Cu at (247.6, 160.6)
- added INTERRUPT_GPIO2: SW_Push, Connector_Wire:SolderWire-0.1sqmm_1x02_P3.6mm_D0.4mm_OD1mm, B.Cu at (98.6, 19.1)
- added INTERRUPT_GPIO3: SW_Push, Connector_Wire:SolderWire-0.1sqmm_1x02_P3.6mm_D0.4mm_OD1mm, B.Cu at (163.6, 19.1)
- added INTERRUPT_GPIO4: SW_Push, Connector_Wire:SolderWire-0.1sqmm_1x02_P3.6mm_D0.4mm_OD1mm, B.Cu at (228.6, 19.1)
- added INTERRUPT_GPIO5: SW_Push, Connector_Wire:SolderWire-0.1sqmm_1x02_P3.6mm_D0.4mm_OD1mm, B.Cu at (33.6, 99.1)
- added INTERRUPT_GPIO6: SW_Push, Connector_Wire:SolderWire-0.1sqmm_1x02_P3.6mm_D0.4mm_OD1mm, B.Cu at (98.6, 99.1)
- added INTERRUPT_GPIO7: SW_Push, Connector_Wire:SolderWire-0.1sqmm_1x02_P3.6mm_D0.4mm_OD1mm, B.Cu at (163.6, 99.1)
- added INTERRUPT_GPIO8: SW_Push, Connector_Wire:SolderWire-0.1sqmm_1x02_P3.6mm_D0.4mm_OD1mm, B.Cu at (228.6, 99.1)
- added OLED_PINS2: Conn_01x04_Female, Connector_Wire:SolderWire-0.1sqmm_1x04_P3.6mm_D0.4mm_OD1mm, B.Cu at (120.5, 60.3)
- added OLED_PINS3: Conn_01x04_Female, Connector_Wire:SolderWire-0.1sqmm_1x04_P3.6mm_D0.4mm_OD1mm, B.Cu at (185.5, 60.3)
- added OLED_PINS4: Conn_01x04_Female, Connector_Wire:SolderWire-0.1sqmm_1x04_P3.6mm_D0.4mm_OD1mm, B.Cu at (250.5, 60.3)
- added OLED_PINS5: Conn_01x04_Female, Connector_Wire:SolderWire-0.1sqmm_1x04_P3.6mm_D0.4mm_OD1mm, B.Cu at (55.5, 140.3)
- added OLED_PINS6: Conn_01x04_Female, Connector_Wire:SolderWire-0.1sqmm_1x04_P3.6mm_D0.4mm_OD1mm, B.Cu at (120.5, 140.3)
- added OLED_PINS7: Conn_01x04_Female, Connector_Wire:SolderWire-0.1sqmm_1x04_P3.6mm_D0.4mm_OD1mm, B.Cu at (185.5, 140.3)
- added OLED_PINS8: Conn_01x04_Female, Connector_Wire:SolderWire-0.1sqmm_1x04_P3.6mm_D0.4mm_OD1mm, B.Cu at (250.5, 140.3)
- added R10: 120, Resistor_THT:R_Axial_DIN0204_L3.6mm_D1.6mm_P7.62mm_Horizontal, B.Cu at (60.3, 152.7)
- added R11: 120, Resistor_THT:R_Axial_DIN0204_L3.6mm_D1.6mm_P7.62mm_Horizontal, B.Cu at (96.3, 105.5)
- added R12: 120, Resistor_THT:R_Axial_DIN0204_L3.6mm_D1.6mm_P7.62mm_Horizontal, B.Cu at (125.3, 152.7)
- added R13: 120, Resistor_THT:R_Axial_DIN0204_L3.6mm_D1.6mm_P7.62mm_Horizontal, B.Cu at (161.3, 105.5)
- added R14: 120, Resistor_THT:R_Axial_DIN0204_L3.6mm_D1.6mm_P7.62mm_Horizontal, B.Cu at (190.3, 152.7)
- added R15: 120, Resistor_THT:R_Axial_DIN0204_L3.6mm_D1.6mm_P7.62mm_Horizontal, B.Cu at (226.3, 105.5)
- added R16: 120, Resistor_THT:R_Axial_DIN0204_L3.6mm_D1.6mm_P7.62mm_Horizontal, B.Cu at (255.3, 152.7)
- added R3: 120, Resistor_THT:R_Axial_DIN0204_L3.6mm_D1.6mm_P7.62mm_Horizontal, B.Cu at (96.3, 25.5)
- added R4: 120, Resistor_THT:R_Axial_DIN0204_L3.6mm_D1.6mm_P7.62mm_Horizontal, B.Cu at (125.3, 72.7)
- added R5: 120, Resistor_THT:R_Axial_DIN0204_L3.6mm_D1.6mm_P7.62mm_Horizontal, B.Cu at (161.3, 25.5)
- added R6: 120, Resistor_THT:R_Axial_DIN0204_L3.6mm_D1.6mm_P7.62mm_Horizontal, B.Cu at (190.3, 72.7)
- added R7: 120, Resistor_THT:R_Axial_DIN0204_L3.6mm_D1.6mm_P7.62mm_Horizontal, B.Cu at (226.3, 25.5)
- added R8: 120, Resistor_THT:R_Axial_DIN0204_L3.6mm_D1.6mm_P7.62mm_Horizontal, B.Cu at (255.3, 72.7)
- added R9: 120, Resistor_THT:R_Axial_DIN0204_L3.6mm_D1.6mm_P7.62mm_Horizontal, B.Cu at (31.3, 105.5)
- added REF**1: MountingHole_2.2mm_M2, MountingHole:MountingHole_2.2mm_M2, F.Cu at (92.1, 79.5)
- added REF**10: MountingHole_2.2mm_M2, MountingHole:MountingHole_2.2mm_M2, F.Cu at (270.3, 79.5)
- added REF**11: MountingHole_2.2mm_M2, MountingHole:MountingHole_2.2mm_M2, F.Cu at (222.1, 19.5)
- added REF**12: MountingHole_2.2mm_M2, MountingHole:MountingHole_2.2mm_M2, F.Cu at (270.5, 19.4)
- added REF**13: MountingHole_2.2mm_M2, MountingHole:MountingHole_2.2mm_M2, F.Cu at (27.1, 159.5)
- added REF**14: MountingHole_2.2mm_M2, MountingHole:MountingHole_2.2mm_M2, F.Cu at (75.3, 159.5)
- added REF**15: MountingHole_2.2mm_M2, MountingHole:MountingHole_2.2mm_M2, F.Cu at (27.1, 99.5)
- added REF**16: MountingHole_2.2mm_M2, MountingHole:MountingHole_2.2mm_M2, F.Cu at (75.5, 99.4)
- added REF**17: MountingHole_2.2mm_M2, MountingHole:MountingHole_2.2mm_M2, F.Cu at (92.1, 159.5)
- added REF**18: MountingHole_2.2mm_M2, MountingHole:MountingHole_2.2mm_M2, F.Cu at (140.3, 159.5)
- added REF**19: MountingHole_2.2mm_M2, MountingHole:MountingHole_2.2mm_M2, F.Cu at (92.1, 99.5)
- added REF**2: MountingHole_2.2mm_M2, MountingHole:MountingHole_2.2mm_M2, F.Cu at (140.3, 79.5)
- added REF**20: MountingHole_2.2mm_M2, MountingHole:MountingHole_2.2mm_M2, F.Cu at (140.5, 99.4)
- added REF**21: MountingHole_2.2mm_M2, MountingHole:MountingHole_2.2mm_M2, F.Cu at (157.1, 159.5)
- added REF**22: MountingHole_2.2mm_M2, MountingHole:MountingHole_2.2mm_M2, F.Cu at (205.3, 159.5)
- added REF**23: MountingHole_2.2mm_M2, MountingHole:MountingHole_2.2mm_M2, F.Cu at (157.1, 99.5)
- added REF**24: MountingHole_2.2mm_M2, MountingHole:MountingHole_2.2mm_M2, F.Cu at (205.5, 99.4)
- added REF**25: MountingHole_2.2mm_M2, MountingHole:MountingHole_2.2mm_M2, F.Cu at (222.1, 159.5)
- added REF**26: MountingHole_2.2mm_M2, MountingHole:MountingHole_2.2mm_M2, F.Cu at (270.3, 159.5)
- added REF**27: MountingHole_2.2mm_M2, MountingHole:MountingHole_2.2mm_M2, F.Cu at (222.1, 99.5)
- added REF**28: MountingHole_2.2mm_M2, MountingHole:MountingHole_2.2mm_M2, F.Cu at (270.5, 99.4)
- added REF**3: MountingHole_2.2mm_M2, MountingHole:MountingHole_2.2mm_M2, F.Cu at (92.1, 19.5)
- added REF**4: MountingHole_2.2mm_M2, MountingHole:MountingHole_2.2mm_M2, F.Cu at (140.5, 19.4)
- added REF**5: MountingHole_2.2mm_M2, MountingHole:MountingHole_2.2mm_M2, F.Cu at (157.1, 79.5)
- added REF**6: MountingHole_2.2mm_M2, MountingHole:MountingHole_2.2mm_M2, F.Cu at (205.3, 79.5)
- added REF**7: MountingHole_2.2mm_M2, MountingHole:MountingHole_2.2mm_M2, F.Cu at (157.1, 19.5)
- added REF**8: MountingHole_2.2mm_M2, MountingHole:MountingHole_2.2mm_M2, F.Cu at (205.5, 19.4)
- added REF**9: MountingHole_2.2mm_M2, MountingHole:MountingHole_2.2mm_M2, F.Cu at (222.1, 79.5)
- added SIGNAL_IN2: TestPoint, TestPoint:TestPoint_Keystone_5015_Micro-Minature, B.Cu at (117.9, 19.2)
- added SIGNAL_IN3: TestPoint, TestPoint:TestPoint_Keystone_5015_Micro-Minature, B.Cu at (182.9, 19.2)
- added SIGNAL_IN4: TestPoint, TestPoint:TestPoint_Keystone_5015_Micro-Minature, B.Cu at (247.9, 19.2)
- added SIGNAL_IN5: TestPoint, TestPoint:TestPoint_Keystone_5015_Micro-Minature, B.Cu at (52.9, 99.2)
- added SIGNAL_IN6: TestPoint, TestPoint:TestPoint_Keystone_5015_Micro-Minature, B.Cu at (117.9, 99.2)
- added SIGNAL_IN7: TestPoint, TestPoint:TestPoint_Keystone_5015_Micro-Minature, B.Cu at (182.9, 99.2)
- added SIGNAL_IN8: TestPoint, TestPoint:TestPoint_Keystone_5015_Micro-Minature, B.Cu at (247.9, 99.2)
- added U2: ESP32_DevKit_V1_DOIT, esp32_devkit_v1_doit:esp32_devkit_v1_doit, F.Cu at (116.2, 67.9)
- added U3: ESP32_DevKit_V1_DOIT, esp32_devkit_v1_doit:esp32_devkit_v1_doit, F.Cu at (181.2, 67.9)
- added U4: ESP32_DevKit_V1_DOIT, esp32_devkit_v1_doit:esp32_devkit_v1_doit, F.Cu at (246.2, 67.9)
- added U5: ESP32_DevKit_V1_DOIT, esp32_devkit_v1_doit:esp32_devkit_v1_doit, F.Cu at (51.2, 147.9)
- added U6: ESP32_DevKit_V1_DOIT, esp32_devkit_v1_doit:esp32_devkit_v1_doit, F.Cu at (116.2, 147.9)
- added U7: ESP32_DevKit_V1_DOIT, esp32_devkit_v1_doit:esp32_devkit_v1_doit, F.Cu at (181.2, 147.9)
- added U8: ESP32_DevKit_V1_DOIT, esp32_devkit_v1_doit:esp32_devkit_v1_doit, F.Cu at (246.2, 147.9)
- moved REF** 6.42 mm to (75.3, 79.5)
- moved REF** 6.42 mm to (75.5, 19.4)
- moved REF** 6.42 mm to (27.1, 79.5)
- moved 3V3_OUT1 6.42 mm to (43.6, 19.2)
- moved SIGNAL_IN1 6.42 mm to (52.9, 19.2)
- moved OLED_PINS1 6.42 mm to (55.5, 60.3)
- moved D1 6.42 mm to (52.6, 80.6)
- moved R1 6.42 mm to (31.3, 25.5)
- moved R2 6.42 mm to (60.3, 72.7)
- moved U1 6.42 mm to (51.2, 67.9)
- moved 100nF1 6.42 mm to (55.0, 67.1)
- moved BZ1 6.42 mm to (30.1, 44.7)
- moved INTERRUPT_GPIO1 6.42 mm to (33.6, 19.1)
- moved REF** 6.42 mm to (27.1, 19.5)
- moved BATTERY1 6.42 mm to (62.5, 19.4)
Routing:
- net Net-(100nF1-Pad1): track 52.2 -> 418.0 mm
- net Net-(3V3_OUT1-Pad1): track 47.6 -> 380.9 mm
- net Net-(INTERRUPT_GPIO1-Pad1): track 44.7 -> 357.7 mm
- net Net-(D1-Pad2): track 22.5 -> 179.8 mm
- net Net-(OLED_PINS1-Pad4): track 20.4 -> 163.4 mm
- net Net-(OLED_PINS1-Pad3): track 17.8 -> 142.0 mm
- net Net-(BATTERY1-Pad1): track 13.5 -> 108.3 mm
- net Net-(BZ1-Pad2): track 11.5 -> 92.2 mm
- net Net-(BZ1-Pad1): track 11.5 -> 91.7 mm
- net Net-(D1-Pad1): track 11.1 -> 88.5 mm
- net Net-(100nF1-Pad2): track 8.70 -> 69.6 mm
- net GND: track 0.09 -> 0.70 mm
Other:
- board size 54.8 x 66.9 mm -> 249.8 x 146.9 mm
