File: peripherals/glucometer-pcb.kicad_pcb (KiCad board)
At the start: 2 copper layers, 249.8 x 146.9 mm, 120 parts, among them U1 ESP32_DevKit_V1_DOIT, U2 ESP32_DevKit_V1_DOIT, U3 ESP32_DevKit_V1_DOIT, U4 ESP32_DevKit_V1_DOIT, U5 ESP32_DevKit_V1_DOIT, U6 ESP32_DevKit_V1_DOIT, U7 ESP32_DevKit_V1_DOIT, U8 ESP32_DevKit_V1_DOIT

Commit message: peripherals pcb update
Parts:
- removed 100nF2, 100nF3, 100nF4, 100nF5, 100nF6, 100nF7, 100nF8: CAP, Capacitor_THT:C_Disc_D4.3mm_W1.9mm_P5.00mm
- removed 3V3_OUT2, 3V3_OUT3, 3V3_OUT4, 3V3_OUT5, 3V3_OUT6, 3V3_OUT7, 3V3_OUT8, SIGNAL_IN2, SIGNAL_IN3, SIGNAL_IN4, SIGNAL_IN5, SIGNAL_IN6, SIGNAL_IN7, SIGNAL_IN8: TestPoint, TestPoint:TestPoint_Keystone_5015_Micro-Minature
- removed BATTERY2, BATTERY3, BATTERY4, BATTERY5, BATTERY6, BATTERY7, BATTERY8: Battery_Cell, Connector_Wire:SolderWire-0.1sqmm_1x02_P3.6mm_D0.4mm_OD1mm
- removed BZ2, BZ3, BZ4, BZ5, BZ6, BZ7, BZ8: Buzzer, Buzzer_Beeper:MagneticBuzzer_ProSignal_ABI-009-RC
- removed D2, D3, D4, D5, D6, D7, D8: EMITTER, LED_THT:LED_D3.0mm_Clear
- removed INTERRUPT_GPIO2, INTERRUPT_GPIO3, INTERRUPT_GPIO4, INTERRUPT_GPIO5, INTERRUPT_GPIO6, INTERRUPT_GPIO7, INTERRUPT_GPIO8: SW_Push, Connector_Wire:SolderWire-0.1sqmm_1x02_P3.6mm_D0.4mm_OD1mm
- removed OLED_PINS1, OLED_PINS2, OLED_PINS3, OLED_PINS4, OLED_PINS5, OLED_PINS6, OLED_PINS7, OLED_PINS8: Conn_01x04_Female, Connector_Wire:SolderWire-0.1sqmm_1x04_P3.6mm_D0.4mm_OD1mm
- removed R10, R11, R12, R13, R14, R15, R16, R3, R4, R5, R6, R7, R8, R9: 120, Resistor_THT:R_Axial_DIN0204_L3.6mm_D1.6mm_P7.62mm_Horizontal
- removed REF**1, REF**10, REF**11, REF**12, REF**13, REF**14, REF**15, REF**16, REF**17, REF**18, REF**19, REF**2, REF**20, REF**21, REF**22, REF**23, REF**24, REF**25, REF**26, REF**27, REF**28, REF**3, REF**4, REF**5, REF**6, REF**7, REF**8, REF**9: MountingHole_2.2mm_M2, MountingHole:MountingHole_2.2mm_M2
- removed U2, U3, U4, U5, U6, U7, U8: ESP32_DevKit_V1_DOIT, esp32_devkit_v1_doit:esp32_devkit_v1_doit
- added GND1: TestPoint, TestPoint:TestPoint_Pad_2.0x2.0mm, B.Cu at (120.3, 66.4)
- added SCL1: TestPoint, TestPoint:TestPoint_Pad_2.0x2.0mm, B.Cu at (125.6, 66.2)
- added SDA1: TestPoint, TestPoint:TestPoint_Pad_2.0x2.0mm, B.Cu at (125.6, 71.6)
- added VCC1: TestPoint, TestPoint:TestPoint_Pad_2.0x2.0mm, B.Cu at (120.3, 71.7)
- 100nF1, BZ1, R1, R2: moved to F.Cu
- moved REF** 133.1 mm to (154.9, 116.8)
- moved REF** 131.9 mm to (152.4, 60.6)
- moved D1 102.7 mm to (120.7, 157.5)
- moved R1 100.1 mm to (114.5, 81.2), turned to -90 degrees
- moved REF** 98.6 mm to (165.1, 60.5)
- moved REF** 97.2 mm to (165.1, 116.8)
- moved 100nF1 91.7 mm to (136.5, 109.2), turned to -90 degrees
- moved SIGNAL_IN1 89.2 mm to (132.1, 60.4)
- moved U1 86.8 mm to (119.2, 121.9)
- moved 3V3_OUT1 81.8 mm to (114.3, 60.4)
- moved INTERRUPT_GPIO1 81.7 mm to (104.1, 60.3)
- moved BZ1 79.5 mm to (105.8, 69.0), turned to 0 degrees
- moved BATTERY1 74.2 mm to (124.5, 60.2)
- moved R2 72.4 mm to (114.6, 120.7), turned to 90 degrees
Routing:
- net Net-(100nF1-Pad1): track 418.0 -> 50.8 mm
- net Net-(3V3_OUT1-Pad1): track 380.9 -> 42.8 mm
- net Net-(INTERRUPT_GPIO1-Pad1): track 357.7 -> 51.1 mm
- net Net-(D1-Pad2): track 179.8 -> 43.0 mm
- net Net-(SDA1-Pad1): track 163.4 -> 55.7 mm
- net Net-(SCL1-Pad1): track 142.0 -> 53.5 mm
- net Net-(BZ1-Pad2): track 92.2 -> 12.2 mm
- net Net-(BATTERY1-Pad1): track 108.3 -> 29.2 mm
- net Net-(100nF1-Pad2): track 69.6 -> 4.70 mm
- net Net-(BZ1-Pad1): track 91.7 -> 39.1 mm
- net Net-(D1-Pad1): track 88.5 -> 39.4 mm
- net unconnected-(U1-Pad19): track 0.00 -> 0.83 mm
- net GND: track 0.70 -> 0.00 mm
- removed copper zone on B.Cu, net GND
Other:
- board size 249.8 x 146.9 mm -> 54.8 x 102.4 mm

Commit message: pcb update
Parts:
- added 100nF1: CAP, Capacitor_THT:C_Disc_D4.3mm_W1.9mm_P5.00mm, F.Cu at (74.0, 146.6)
- added 100nF1: CAP, Capacitor_THT:C_Disc_D4.3mm_W1.9mm_P5.00mm, F.Cu at (264.8, 69.5)
- added 100nF1: CAP, Capacitor_THT:C_Disc_D4.3mm_W1.9mm_P5.00mm, F.Cu at (129.1, 72.1)
- added 100nF1: CAP, Capacitor_THT:C_Disc_D4.3mm_W1.9mm_P5.00mm, F.Cu at (213.7, 146.6)
- added 100nF1: CAP, Capacitor_THT:C_Disc_D4.3mm_W1.9mm_P5.00mm, F.Cu at (194.8, 70.2)
- added 3V3_OUT1: TestPoint, TestPoint:TestPoint_Keystone_5015_Micro-Minature, B.Cu at (244.7, 20.5)
- added 3V3_OUT1: TestPoint, TestPoint:TestPoint_Keystone_5015_Micro-Minature, B.Cu at (174.7, 21.3)
- added 3V3_OUT1: TestPoint, TestPoint:TestPoint_Keystone_5015_Micro-Minature, B.Cu at (109.0, 23.1)
- added 3V3_OUT1: TestPoint, TestPoint:TestPoint_Keystone_5015_Micro-Minature, B.Cu at (164.7, 166.7)
- added 3V3_OUT1: TestPoint, TestPoint:TestPoint_Keystone_5015_Micro-Minature, B.Cu at (25.0, 166.7)
- added BATTERY1: Battery_Cell, Connector_Wire:SolderWire-0.1sqmm_1x02_P3.6mm_D0.4mm_OD1mm, B.Cu at (25.0, 156.8)
- added BATTERY1: Battery_Cell, Connector_Wire:SolderWire-0.1sqmm_1x02_P3.6mm_D0.4mm_OD1mm, B.Cu at (118.9, 23.1)
- added BATTERY1: Battery_Cell, Connector_Wire:SolderWire-0.1sqmm_1x02_P3.6mm_D0.4mm_OD1mm, B.Cu at (254.6, 20.5)
- added BATTERY1: Battery_Cell, Connector_Wire:SolderWire-0.1sqmm_1x02_P3.6mm_D0.4mm_OD1mm, B.Cu at (164.7, 156.8)
- added BATTERY1: Battery_Cell, Connector_Wire:SolderWire-0.1sqmm_1x02_P3.6mm_D0.4mm_OD1mm, B.Cu at (184.6, 21.3)
- added BZ1: Buzzer, Buzzer_Beeper:MagneticBuzzer_ProSignal_ABI-009-RC, F.Cu at (33.7, 179.3)
- added BZ1: Buzzer, Buzzer_Beeper:MagneticBuzzer_ProSignal_ABI-009-RC, F.Cu at (96.5, 31.8)
- added BZ1: Buzzer, Buzzer_Beeper:MagneticBuzzer_ProSignal_ABI-009-RC, F.Cu at (173.4, 179.3)
- added BZ1: Buzzer, Buzzer_Beeper:MagneticBuzzer_ProSignal_ABI-009-RC, F.Cu at (232.2, 29.2)
- added BZ1: Buzzer, Buzzer_Beeper:MagneticBuzzer_ProSignal_ABI-009-RC, F.Cu at (162.2, 30.0)
- added D1: EMITTER, LED_THT:LED_D3.0mm_Clear, F.Cu at (120.5, 161.5)
- added D1: EMITTER, LED_THT:LED_D3.0mm_Clear, F.Cu at (260.3, 161.5)
- added D1: EMITTER, LED_THT:LED_D3.0mm_Clear, F.Cu at (179.9, 116.8)
- added D1: EMITTER, LED_THT:LED_D3.0mm_Clear, F.Cu at (114.2, 118.6)
- added D1: EMITTER, LED_THT:LED_D3.0mm_Clear, F.Cu at (249.9, 116.0)
- added GND1: TestPoint, TestPoint:TestPoint_Pad_2.0x2.0mm, B.Cu at (167.8, 35.9)
- added GND1: TestPoint, TestPoint:TestPoint_Pad_2.0x2.0mm, B.Cu at (102.1, 37.7)
- added GND1: TestPoint, TestPoint:TestPoint_Pad_2.0x2.0mm, B.Cu at (179.3, 173.6)
- added GND1: TestPoint, TestPoint:TestPoint_Pad_2.0x2.0mm, B.Cu at (237.8, 35.1)
- added GND1: TestPoint, TestPoint:TestPoint_Pad_2.0x2.0mm, B.Cu at (39.6, 173.6)
- added INTERRUPT_GPIO1: SW_Push, Connector_Wire:SolderWire-0.1sqmm_1x02_P3.6mm_D0.4mm_OD1mm, B.Cu at (233.7, 20.5)
- added INTERRUPT_GPIO1: SW_Push, Connector_Wire:SolderWire-0.1sqmm_1x02_P3.6mm_D0.4mm_OD1mm, B.Cu at (163.8, 21.3)
- added INTERRUPT_GPIO1: SW_Push, Connector_Wire:SolderWire-0.1sqmm_1x02_P3.6mm_D0.4mm_OD1mm, B.Cu at (25.0, 177.7)
- added INTERRUPT_GPIO1: SW_Push, Connector_Wire:SolderWire-0.1sqmm_1x02_P3.6mm_D0.4mm_OD1mm, B.Cu at (164.7, 177.7)
- added INTERRUPT_GPIO1: SW_Push, Connector_Wire:SolderWire-0.1sqmm_1x02_P3.6mm_D0.4mm_OD1mm, B.Cu at (98.0, 23.1)
- added R1: 120, Resistor_THT:R_Axial_DIN0204_L3.6mm_D1.6mm_P7.62mm_Horizontal, F.Cu at (33.8, 158.3)
- added R1: 120, Resistor_THT:R_Axial_DIN0204_L3.6mm_D1.6mm_P7.62mm_Horizontal, F.Cu at (117.4, 31.9)
- added R1: 120, Resistor_THT:R_Axial_DIN0204_L3.6mm_D1.6mm_P7.62mm_Horizontal, F.Cu at (183.1, 30.1)
- added R1: 120, Resistor_THT:R_Axial_DIN0204_L3.6mm_D1.6mm_P7.62mm_Horizontal, F.Cu at (253.1, 29.3)
- added R1: 120, Resistor_THT:R_Axial_DIN0204_L3.6mm_D1.6mm_P7.62mm_Horizontal, F.Cu at (173.5, 158.3)
- added R2: 120, Resistor_THT:R_Axial_DIN0204_L3.6mm_D1.6mm_P7.62mm_Horizontal, F.Cu at (85.4, 168.5)
- added R2: 120, Resistor_THT:R_Axial_DIN0204_L3.6mm_D1.6mm_P7.62mm_Horizontal, F.Cu at (225.1, 168.5)
- added R2: 120, Resistor_THT:R_Axial_DIN0204_L3.6mm_D1.6mm_P7.62mm_Horizontal, F.Cu at (173.0, 81.7)
- added R2: 120, Resistor_THT:R_Axial_DIN0204_L3.6mm_D1.6mm_P7.62mm_Horizontal, F.Cu at (107.3, 83.5)
- added R2: 120, Resistor_THT:R_Axial_DIN0204_L3.6mm_D1.6mm_P7.62mm_Horizontal, F.Cu at (243.0, 80.9)
- added REF**: MountingHole_2.2mm_M2, MountingHole:MountingHole_2.2mm_M2, F.Cu at (261.0, 142.9)
- added REF**: MountingHole_2.2mm_M2, MountingHole:MountingHole_2.2mm_M2, F.Cu at (164.3, 182.6)
- added REF**: MountingHole_2.2mm_M2, MountingHole:MountingHole_2.2mm_M2, F.Cu at (198.4, 21.0)
- added REF**: MountingHole_2.2mm_M2, MountingHole:MountingHole_2.2mm_M2, F.Cu at (121.2, 142.9)
- added REF**: MountingHole_2.2mm_M2, MountingHole:MountingHole_2.2mm_M2, F.Cu at (24.8, 143.0)
- added REF**: MountingHole_2.2mm_M2, MountingHole:MountingHole_2.2mm_M2, F.Cu at (261.0, 182.8)
- added REF**: MountingHole_2.2mm_M2, MountingHole:MountingHole_2.2mm_M2, F.Cu at (228.7, 116.8)
- added REF**: MountingHole_2.2mm_M2, MountingHole:MountingHole_2.2mm_M2, F.Cu at (158.8, 20.9)
- added REF**: MountingHole_2.2mm_M2, MountingHole:MountingHole_2.2mm_M2, F.Cu at (164.5, 143.0)
- added REF**: MountingHole_2.2mm_M2, MountingHole:MountingHole_2.2mm_M2, F.Cu at (93.0, 119.4)
- added REF**: MountingHole_2.2mm_M2, MountingHole:MountingHole_2.2mm_M2, F.Cu at (228.8, 20.1)
- added REF**: MountingHole_2.2mm_M2, MountingHole:MountingHole_2.2mm_M2, F.Cu at (198.5, 117.5)
- added REF**: MountingHole_2.2mm_M2, MountingHole:MountingHole_2.2mm_M2, F.Cu at (158.7, 117.6)
- added REF**: MountingHole_2.2mm_M2, MountingHole:MountingHole_2.2mm_M2, F.Cu at (268.4, 20.3)
- added REF**: MountingHole_2.2mm_M2, MountingHole:MountingHole_2.2mm_M2, F.Cu at (132.7, 22.9)
- added REF**: MountingHole_2.2mm_M2, MountingHole:MountingHole_2.2mm_M2, F.Cu at (24.6, 182.6)
- added REF**: MountingHole_2.2mm_M2, MountingHole:MountingHole_2.2mm_M2, F.Cu at (121.3, 182.8)
- added REF**: MountingHole_2.2mm_M2, MountingHole:MountingHole_2.2mm_M2, F.Cu at (268.5, 116.8)
- added REF**: MountingHole_2.2mm_M2, MountingHole:MountingHole_2.2mm_M2, F.Cu at (132.8, 119.3)
- added REF**: MountingHole_2.2mm_M2, MountingHole:MountingHole_2.2mm_M2, F.Cu at (93.1, 22.7)
- added SCL1: TestPoint, TestPoint:TestPoint_Pad_2.0x2.0mm, B.Cu at (39.6, 160.5)
- added SCL1: TestPoint, TestPoint:TestPoint_Pad_2.0x2.0mm, B.Cu at (179.3, 160.5)
- added SCL1: TestPoint, TestPoint:TestPoint_Pad_2.0x2.0mm, B.Cu at (180.9, 35.9)
- added SCL1: TestPoint, TestPoint:TestPoint_Pad_2.0x2.0mm, B.Cu at (115.2, 37.7)
- added SCL1: TestPoint, TestPoint:TestPoint_Pad_2.0x2.0mm, B.Cu at (250.9, 35.1)
- added SDA1: TestPoint, TestPoint:TestPoint_Pad_2.0x2.0mm, B.Cu at (179.3, 154.0)
- added SDA1: TestPoint, TestPoint:TestPoint_Pad_2.0x2.0mm, B.Cu at (187.4, 35.9)
- added SDA1: TestPoint, TestPoint:TestPoint_Pad_2.0x2.0mm, B.Cu at (121.7, 37.7)
- added SDA1: TestPoint, TestPoint:TestPoint_Pad_2.0x2.0mm, B.Cu at (39.6, 154.0)
- added SDA1: TestPoint, TestPoint:TestPoint_Pad_2.0x2.0mm, B.Cu at (257.4, 35.1)
- added SIGNAL_IN1: TestPoint, TestPoint:TestPoint_Keystone_5015_Micro-Minature, B.Cu at (164.8, 149.1)
- added SIGNAL_IN1: TestPoint, TestPoint:TestPoint_Keystone_5015_Micro-Minature, B.Cu at (192.3, 21.4)
- added SIGNAL_IN1: TestPoint, TestPoint:TestPoint_Keystone_5015_Micro-Minature, B.Cu at (262.3, 20.6)
- added SIGNAL_IN1: TestPoint, TestPoint:TestPoint_Keystone_5015_Micro-Minature, B.Cu at (126.6, 23.2)
- added SIGNAL_IN1: TestPoint, TestPoint:TestPoint_Keystone_5015_Micro-Minature, B.Cu at (25.1, 149.1)
- added U1: ESP32_DevKit_V1_DOIT, esp32_devkit_v1_doit:esp32_devkit_v1_doit, F.Cu at (111.9, 84.8)
- added U1: ESP32_DevKit_V1_DOIT, esp32_devkit_v1_doit:esp32_devkit_v1_doit, F.Cu at (86.7, 163.9)
- added U1: ESP32_DevKit_V1_DOIT, esp32_devkit_v1_doit:esp32_devkit_v1_doit, F.Cu at (177.6, 83.0)
- added U1: ESP32_DevKit_V1_DOIT, esp32_devkit_v1_doit:esp32_devkit_v1_doit, F.Cu at (226.4, 163.9)
- added U1: ESP32_DevKit_V1_DOIT, esp32_devkit_v1_doit:esp32_devkit_v1_doit, F.Cu at (247.6, 82.2)
- added VCC1: TestPoint, TestPoint:TestPoint_Pad_2.0x2.0mm, B.Cu at (108.7, 37.7)
- added VCC1: TestPoint, TestPoint:TestPoint_Pad_2.0x2.0mm, B.Cu at (179.3, 167.1)
- added VCC1: TestPoint, TestPoint:TestPoint_Pad_2.0x2.0mm, B.Cu at (39.6, 167.1)
- added VCC1: TestPoint, TestPoint:TestPoint_Pad_2.0x2.0mm, B.Cu at (174.4, 35.9)
- added VCC1: TestPoint, TestPoint:TestPoint_Pad_2.0x2.0mm, B.Cu at (244.4, 35.1)
- moved REF** 158.9 mm to (26.2, 23.6)
- moved REF** 139.0 mm to (26.1, 120.4)
- moved REF** 115.7 mm to (66.0, 120.3)
- moved REF** 94.1 mm to (65.8, 23.8)
- moved GND1 89.5 mm to (35.3, 38.7)
- moved VCC1 85.2 mm to (41.8, 38.7)
- moved BZ1 84.4 mm to (29.6, 32.7)
- moved 100nF1 82.5 mm to (62.3, 73.0)
- moved R2 82.5 mm to (40.4, 84.5)
- moved U1 82.5 mm to (45.0, 85.7)
- moved D1 82.5 mm to (47.4, 119.6)
- moved SCL1 82.1 mm to (48.3, 38.7)
- moved INTERRUPT_GPIO1 81.4 mm to (31.2, 24.0)
- moved BATTERY1 80.9 mm to (52.1, 24.0)
- moved SIGNAL_IN1 80.9 mm to (59.8, 24.1)
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Routing:
- net Net-(SDA1-Pad1): track 55.7 -> 350.9 mm
- net Net-(SCL1-Pad1): track 53.5 -> 329.7 mm
- net Net-(INTERRUPT_GPIO1-Pad1): track 51.1 -> 319.2 mm
- net Net-(100nF1-Pad1): track 50.8 -> 299.9 mm
- net Net-(D1-Pad2): track 43.0 -> 250.0 mm
- net Net-(3V3_OUT1-Pad1): track 42.8 -> 246.6 mm
- net Net-(BZ1-Pad1): track 39.1 -> 234.8 mm
- net Net-(D1-Pad1): track 39.4 -> 228.1 mm
- net Net-(BATTERY1-Pad1): track 29.2 -> 197.6 mm
- net Net-(BZ1-Pad2): track 12.2 -> 73.8 mm
- net Net-(100nF1-Pad2): track 4.70 -> 28.2 mm
- net unconnected-(U1-Pad19): track 0.83 -> 0.00 mm
- added copper zone on B.Cu, net GND
Other:
- board size 54.8 x 102.4 mm -> 250.4 x 169.2 mm

Commit message: asd
Parts:
- removed the 100nF1 at (74.0, 146.6)
- removed the 100nF1 at (264.8, 69.5)
- removed the 100nF1 at (129.1, 72.1)
- removed the 100nF1 at (213.7, 146.6)
- removed the 100nF1 at (194.8, 70.2)
- removed the 3V3_OUT1 at (244.7, 20.5)
- removed the 3V3_OUT1 at (174.7, 21.3)
- removed the 3V3_OUT1 at (109.0, 23.1)
- removed the 3V3_OUT1 at (164.7, 166.7)
- removed the 3V3_OUT1 at (25.0, 166.7)
- removed the BATTERY1 at (25.0, 156.8)
- removed the BATTERY1 at (118.9, 23.1)
- removed the BATTERY1 at (254.6, 20.5)
- removed the BATTERY1 at (164.7, 156.8)
- removed the BATTERY1 at (184.6, 21.3)
- removed the BZ1 at (33.7, 179.3)
- removed the BZ1 at (96.5, 31.8)
- removed the BZ1 at (173.4, 179.3)
- removed the BZ1 at (232.2, 29.2)
- removed the BZ1 at (162.2, 30.0)
- removed the D1 at (120.5, 161.5)
- removed the D1 at (260.3, 161.5)
- removed the D1 at (179.9, 116.8)
- removed the D1 at (114.2, 118.6)
- removed the D1 at (249.9, 116.0)
- removed the GND1 at (167.8, 35.9)
- removed the GND1 at (102.1, 37.7)
- removed the GND1 at (179.3, 173.6)
- removed the GND1 at (237.8, 35.1)
- removed the GND1 at (39.6, 173.6)
- removed the INTERRUPT_GPIO1 at (233.7, 20.5)
- removed the INTERRUPT_GPIO1 at (163.8, 21.3)
- removed the INTERRUPT_GPIO1 at (25.0, 177.7)
- removed the INTERRUPT_GPIO1 at (164.7, 177.7)
- removed the INTERRUPT_GPIO1 at (98.0, 23.1)
- removed the R1 at (33.8, 158.3)
- removed the R1 at (117.4, 31.9)
- removed the R1 at (183.1, 30.1)
- removed the R1 at (253.1, 29.3)
- removed the R1 at (173.5, 158.3)
- removed the R2 at (85.4, 168.5)
- removed the R2 at (225.1, 168.5)
- removed the R2 at (173.0, 81.7)
- removed the R2 at (107.3, 83.5)
- removed the R2 at (243.0, 80.9)
- removed the REF** at (261.0, 142.9)
- removed the REF** at (164.3, 182.6)
- removed the REF** at (198.4, 21.0)
- removed the REF** at (121.2, 142.9)
- removed the REF** at (24.8, 143.0)
- removed the REF** at (261.0, 182.8)
- removed the REF** at (228.7, 116.8)
- removed the REF** at (158.8, 20.9)
- removed the REF** at (164.5, 143.0)
- removed the REF** at (93.0, 119.4)
- removed the REF** at (228.8, 20.1)
- removed the REF** at (198.5, 117.5)
- removed the REF** at (158.7, 117.6)
- removed the REF** at (268.4, 20.3)
- removed the REF** at (132.7, 22.9)
- removed the REF** at (24.6, 182.6)
- removed the REF** at (121.3, 182.8)
- removed the REF** at (268.5, 116.8)
- removed the REF** at (132.8, 119.3)
- removed the REF** at (93.1, 22.7)
- removed the SCL1 at (39.6, 160.5)
- removed the SCL1 at (179.3, 160.5)
- removed the SCL1 at (180.9, 35.9)
- removed the SCL1 at (115.2, 37.7)
- removed the SCL1 at (250.9, 35.1)
- removed the SDA1 at (179.3, 154.0)
- removed the SDA1 at (187.4, 35.9)
- removed the SDA1 at (121.7, 37.7)
- removed the SDA1 at (39.6, 154.0)
- removed the SDA1 at (257.4, 35.1)
- removed the SIGNAL_IN1 at (164.8, 149.1)
- removed the SIGNAL_IN1 at (192.3, 21.4)
- removed the SIGNAL_IN1 at (262.3, 20.6)
- removed the SIGNAL_IN1 at (126.6, 23.2)
- removed the SIGNAL_IN1 at (25.1, 149.1)
- removed the U1 at (111.9, 84.8)
- removed the U1 at (86.7, 163.9)
- removed the U1 at (177.6, 83.0)
- removed the U1 at (226.4, 163.9)
- removed the U1 at (247.6, 82.2)
- removed the VCC1 at (108.7, 37.7)
- removed the VCC1 at (179.3, 167.1)
- removed the VCC1 at (39.6, 167.1)
- removed the VCC1 at (174.4, 35.9)
- removed the VCC1 at (244.4, 35.1)
- added 100nF1: CAP, Capacitor_THT:C_Disc_D4.3mm_W1.9mm_P5.00mm, F.Cu at (125.2, 73.0)
- added 100nF1: CAP, Capacitor_THT:C_Disc_D4.3mm_W1.9mm_P5.00mm, F.Cu at (212.7, 146.6)
- added 100nF1: CAP, Capacitor_THT:C_Disc_D4.3mm_W1.9mm_P5.00mm, F.Cu at (262.3, 75.5)
- added 100nF1: CAP, Capacitor_THT:C_Disc_D4.3mm_W1.9mm_P5.00mm, F.Cu at (191.2, 73.0)
- added 100nF1: CAP, Capacitor_THT:C_Disc_D4.3mm_W1.9mm_P5.00mm, F.Cu at (75.5, 146.6)
- added 3V3_OUT1: TestPoint, TestPoint:TestPoint_Keystone_5015_Micro-Minature, B.Cu at (171.1, 24.0)
- added 3V3_OUT1: TestPoint, TestPoint:TestPoint_Keystone_5015_Micro-Minature, B.Cu at (163.7, 166.7)
- added 3V3_OUT1: TestPoint, TestPoint:TestPoint_Keystone_5015_Micro-Minature, B.Cu at (105.0, 24.0)
- added 3V3_OUT1: TestPoint, TestPoint:TestPoint_Keystone_5015_Micro-Minature, B.Cu at (242.2, 26.6)
- added 3V3_OUT1: TestPoint, TestPoint:TestPoint_Keystone_5015_Micro-Minature, B.Cu at (26.6, 166.7)
- added BATTERY1: Battery_Cell, Connector_Wire:SolderWire-0.1sqmm_1x02_P3.6mm_D0.4mm_OD1mm, B.Cu at (181.0, 24.0)
- added BATTERY1: Battery_Cell, Connector_Wire:SolderWire-0.1sqmm_1x02_P3.6mm_D0.4mm_OD1mm, B.Cu at (163.7, 156.8)
- added BATTERY1: Battery_Cell, Connector_Wire:SolderWire-0.1sqmm_1x02_P3.6mm_D0.4mm_OD1mm, B.Cu at (26.6, 156.8)
- added BATTERY1: Battery_Cell, Connector_Wire:SolderWire-0.1sqmm_1x02_P3.6mm_D0.4mm_OD1mm, B.Cu at (115.0, 24.0)
- added BATTERY1: Battery_Cell, Connector_Wire:SolderWire-0.1sqmm_1x02_P3.6mm_D0.4mm_OD1mm, B.Cu at (252.1, 26.6)
- added BZ1: Buzzer, Buzzer_Beeper:MagneticBuzzer_ProSignal_ABI-009-RC, F.Cu at (172.4, 179.3)
- added BZ1: Buzzer, Buzzer_Beeper:MagneticBuzzer_ProSignal_ABI-009-RC, F.Cu at (158.5, 32.7)
- added BZ1: Buzzer, Buzzer_Beeper:MagneticBuzzer_ProSignal_ABI-009-RC, F.Cu at (35.3, 179.3)
- added BZ1: Buzzer, Buzzer_Beeper:MagneticBuzzer_ProSignal_ABI-009-RC, F.Cu at (229.7, 35.3)
- added BZ1: Buzzer, Buzzer_Beeper:MagneticBuzzer_ProSignal_ABI-009-RC, F.Cu at (92.5, 32.7)
- added D1: EMITTER, LED_THT:LED_D3.0mm_Clear, F.Cu at (247.4, 122.1)
- added D1: EMITTER, LED_THT:LED_D3.0mm_Clear, F.Cu at (259.3, 161.5)
- added D1: EMITTER, LED_THT:LED_D3.0mm_Clear, F.Cu at (110.3, 119.6)
- added D1: EMITTER, LED_THT:LED_D3.0mm_Clear, F.Cu at (176.3, 119.6)
- added D1: EMITTER, LED_THT:LED_D3.0mm_Clear, F.Cu at (122.1, 161.5)
- added GND1: TestPoint, TestPoint:TestPoint_Pad_2.0x2.0mm, B.Cu at (41.2, 173.6)
- added GND1: TestPoint, TestPoint:TestPoint_Pad_2.0x2.0mm, B.Cu at (98.2, 38.7)
- added GND1: TestPoint, TestPoint:TestPoint_Pad_2.0x2.0mm, B.Cu at (178.4, 173.6)
- added GND1: TestPoint, TestPoint:TestPoint_Pad_2.0x2.0mm, B.Cu at (164.2, 38.7)
- added GND1: TestPoint, TestPoint:TestPoint_Pad_2.0x2.0mm, B.Cu at (235.3, 41.2)
- added INTERRUPT_GPIO1: SW_Push, Connector_Wire:SolderWire-0.1sqmm_1x02_P3.6mm_D0.4mm_OD1mm, B.Cu at (26.6, 177.7)
- added INTERRUPT_GPIO1: SW_Push, Connector_Wire:SolderWire-0.1sqmm_1x02_P3.6mm_D0.4mm_OD1mm, B.Cu at (94.1, 24.0)
- added INTERRUPT_GPIO1: SW_Push, Connector_Wire:SolderWire-0.1sqmm_1x02_P3.6mm_D0.4mm_OD1mm, B.Cu at (231.3, 26.6)
- added INTERRUPT_GPIO1: SW_Push, Connector_Wire:SolderWire-0.1sqmm_1x02_P3.6mm_D0.4mm_OD1mm, B.Cu at (163.7, 177.7)
- added INTERRUPT_GPIO1: SW_Push, Connector_Wire:SolderWire-0.1sqmm_1x02_P3.6mm_D0.4mm_OD1mm, B.Cu at (160.1, 24.0)
- added R1: 120, Resistor_THT:R_Axial_DIN0204_L3.6mm_D1.6mm_P7.62mm_Horizontal, F.Cu at (35.4, 158.3)
- added R1: 120, Resistor_THT:R_Axial_DIN0204_L3.6mm_D1.6mm_P7.62mm_Horizontal, F.Cu at (250.6, 35.4)
- added R1: 120, Resistor_THT:R_Axial_DIN0204_L3.6mm_D1.6mm_P7.62mm_Horizontal, F.Cu at (113.5, 32.8)
- added R1: 120, Resistor_THT:R_Axial_DIN0204_L3.6mm_D1.6mm_P7.62mm_Horizontal, F.Cu at (172.5, 158.3)
- added R1: 120, Resistor_THT:R_Axial_DIN0204_L3.6mm_D1.6mm_P7.62mm_Horizontal, F.Cu at (179.5, 32.8)
- added R2: 120, Resistor_THT:R_Axial_DIN0204_L3.6mm_D1.6mm_P7.62mm_Horizontal, F.Cu at (229.9, 146.7)
- added R2: 120, Resistor_THT:R_Axial_DIN0204_L3.6mm_D1.6mm_P7.62mm_Horizontal, F.Cu at (92.8, 146.7)
- added R2: 120, Resistor_THT:R_Axial_DIN0204_L3.6mm_D1.6mm_P7.62mm_Horizontal, F.Cu at (262.2, 92.8)
- added R2: 120, Resistor_THT:R_Axial_DIN0204_L3.6mm_D1.6mm_P7.62mm_Horizontal, F.Cu at (191.1, 90.2)
- added R2: 120, Resistor_THT:R_Axial_DIN0204_L3.6mm_D1.6mm_P7.62mm_Horizontal, F.Cu at (125.1, 90.2)
- added REF**: MountingHole_2.2mm_M2, MountingHole:MountingHole_2.2mm_M2, F.Cu at (155.2, 23.6)
- added REF**: MountingHole_2.2mm_M2, MountingHole:MountingHole_2.2mm_M2, F.Cu at (128.9, 120.3)
- added REF**: MountingHole_2.2mm_M2, MountingHole:MountingHole_2.2mm_M2, F.Cu at (226.3, 26.2)
- added REF**: MountingHole_2.2mm_M2, MountingHole:MountingHole_2.2mm_M2, F.Cu at (26.3, 143.0)
- added REF**: MountingHole_2.2mm_M2, MountingHole:MountingHole_2.2mm_M2, F.Cu at (265.9, 26.3)
- added REF**: MountingHole_2.2mm_M2, MountingHole:MountingHole_2.2mm_M2, F.Cu at (194.8, 23.8)
- added REF**: MountingHole_2.2mm_M2, MountingHole:MountingHole_2.2mm_M2, F.Cu at (155.1, 120.4)
- added REF**: MountingHole_2.2mm_M2, MountingHole:MountingHole_2.2mm_M2, F.Cu at (163.5, 143.0)
- added REF**: MountingHole_2.2mm_M2, MountingHole:MountingHole_2.2mm_M2, F.Cu at (163.3, 182.6)
- added REF**: MountingHole_2.2mm_M2, MountingHole:MountingHole_2.2mm_M2, F.Cu at (194.9, 120.3)
- added REF**: MountingHole_2.2mm_M2, MountingHole:MountingHole_2.2mm_M2, F.Cu at (260.0, 142.9)
- added REF**: MountingHole_2.2mm_M2, MountingHole:MountingHole_2.2mm_M2, F.Cu at (122.9, 182.8)
- added REF**: MountingHole_2.2mm_M2, MountingHole:MountingHole_2.2mm_M2, F.Cu at (266.0, 122.8)
- added REF**: MountingHole_2.2mm_M2, MountingHole:MountingHole_2.2mm_M2, F.Cu at (128.7, 23.8)
- added REF**: MountingHole_2.2mm_M2, MountingHole:MountingHole_2.2mm_M2, F.Cu at (226.2, 122.9)
- added REF**: MountingHole_2.2mm_M2, MountingHole:MountingHole_2.2mm_M2, F.Cu at (26.2, 182.6)
- added REF**: MountingHole_2.2mm_M2, MountingHole:MountingHole_2.2mm_M2, F.Cu at (89.1, 23.6)
- added REF**: MountingHole_2.2mm_M2, MountingHole:MountingHole_2.2mm_M2, F.Cu at (122.8, 142.9)
- added REF**: MountingHole_2.2mm_M2, MountingHole:MountingHole_2.2mm_M2, F.Cu at (260.1, 182.8)
- added REF**: MountingHole_2.2mm_M2, MountingHole:MountingHole_2.2mm_M2, F.Cu at (89.0, 120.4)
- added SCL1: TestPoint, TestPoint:TestPoint_Pad_2.0x2.0mm, B.Cu at (177.3, 38.7)
- added SCL1: TestPoint, TestPoint:TestPoint_Pad_2.0x2.0mm, B.Cu at (248.4, 41.2)
- added SCL1: TestPoint, TestPoint:TestPoint_Pad_2.0x2.0mm, B.Cu at (178.4, 160.5)
- added SCL1: TestPoint, TestPoint:TestPoint_Pad_2.0x2.0mm, B.Cu at (41.2, 160.5)
- added SCL1: TestPoint, TestPoint:TestPoint_Pad_2.0x2.0mm, B.Cu at (111.2, 38.7)
- added SDA1: TestPoint, TestPoint:TestPoint_Pad_2.0x2.0mm, B.Cu at (41.2, 154.0)
- added SDA1: TestPoint, TestPoint:TestPoint_Pad_2.0x2.0mm, B.Cu at (254.9, 41.2)
- added SDA1: TestPoint, TestPoint:TestPoint_Pad_2.0x2.0mm, B.Cu at (183.8, 38.7)
- added SDA1: TestPoint, TestPoint:TestPoint_Pad_2.0x2.0mm, B.Cu at (178.4, 154.0)
- added SDA1: TestPoint, TestPoint:TestPoint_Pad_2.0x2.0mm, B.Cu at (117.7, 38.7)
- added SIGNAL_IN1: TestPoint, TestPoint:TestPoint_Keystone_5015_Micro-Minature, B.Cu at (163.8, 149.1)
- added SIGNAL_IN1: TestPoint, TestPoint:TestPoint_Keystone_5015_Micro-Minature, B.Cu at (259.8, 26.7)
- added SIGNAL_IN1: TestPoint, TestPoint:TestPoint_Keystone_5015_Micro-Minature, B.Cu at (122.6, 24.1)
- added SIGNAL_IN1: TestPoint, TestPoint:TestPoint_Keystone_5015_Micro-Minature, B.Cu at (26.7, 149.1)
- added SIGNAL_IN1: TestPoint, TestPoint:TestPoint_Keystone_5015_Micro-Minature, B.Cu at (188.7, 24.1)
- added U1: ESP32_DevKit_V1_DOIT, esp32_devkit_v1_doit:esp32_devkit_v1_doit, F.Cu at (173.9, 85.7)
- added U1: ESP32_DevKit_V1_DOIT, esp32_devkit_v1_doit:esp32_devkit_v1_doit, F.Cu at (245.1, 88.3)
- added U1: ESP32_DevKit_V1_DOIT, esp32_devkit_v1_doit:esp32_devkit_v1_doit, F.Cu at (88.3, 163.9)
- added U1: ESP32_DevKit_V1_DOIT, esp32_devkit_v1_doit:esp32_devkit_v1_doit, F.Cu at (225.4, 163.9)
- added U1: ESP32_DevKit_V1_DOIT, esp32_devkit_v1_doit:esp32_devkit_v1_doit, F.Cu at (107.9, 85.7)
- added VCC1: TestPoint, TestPoint:TestPoint_Pad_2.0x2.0mm, B.Cu at (104.7, 38.7)
- added VCC1: TestPoint, TestPoint:TestPoint_Pad_2.0x2.0mm, B.Cu at (241.9, 41.2)
- added VCC1: TestPoint, TestPoint:TestPoint_Pad_2.0x2.0mm, B.Cu at (178.4, 167.1)
- added VCC1: TestPoint, TestPoint:TestPoint_Pad_2.0x2.0mm, B.Cu at (41.2, 167.1)
- added VCC1: TestPoint, TestPoint:TestPoint_Pad_2.0x2.0mm, B.Cu at (170.7, 38.7)
- moved R2 22.5 mm to (62.2, 90.3)
Routing:
- net Net-(SCL1-Pad1): track 329.7 -> 264.3 mm
- net Net-(SDA1-Pad1): track 350.9 -> 325.7 mm
- net Net-(D1-Pad1): track 228.1 -> 213.0 mm
Other:
- board size 250.4 x 169.2 mm -> 246.4 x 165.7 mm

Commit message: emmiter update
Parts:
- removed the 100nF1 at (125.2, 73.0)
- removed the 100nF1 at (212.7, 146.6)
- removed the 100nF1 at (262.3, 75.5)
- removed the 100nF1 at (191.2, 73.0)
- removed the 100nF1 at (75.5, 146.6)
- removed the 3V3_OUT1 at (171.1, 24.0)
- removed the 3V3_OUT1 at (163.7, 166.7)
- removed the 3V3_OUT1 at (105.0, 24.0)
- removed the 3V3_OUT1 at (242.2, 26.6)
- removed the 3V3_OUT1 at (26.6, 166.7)
- removed the BATTERY1 at (181.0, 24.0)
- removed the BATTERY1 at (163.7, 156.8)
- removed the BATTERY1 at (26.6, 156.8)
- removed the BATTERY1 at (115.0, 24.0)
- removed the BATTERY1 at (252.1, 26.6)
- removed the BZ1 at (172.4, 179.3)
- removed the BZ1 at (158.5, 32.7)
- removed the BZ1 at (35.3, 179.3)
- removed the BZ1 at (229.7, 35.3)
- removed the BZ1 at (92.5, 32.7)
- removed the D1 at (247.4, 122.1)
- removed the D1 at (259.3, 161.5)
- removed the D1 at (110.3, 119.6)
- removed the D1 at (176.3, 119.6)
- removed the D1 at (122.1, 161.5)
- removed the GND1 at (41.2, 173.6)
- removed the GND1 at (98.2, 38.7)
- removed the GND1 at (178.4, 173.6)
- removed the GND1 at (164.2, 38.7)
- removed the GND1 at (235.3, 41.2)
- removed the INTERRUPT_GPIO1 at (26.6, 177.7)
- removed the INTERRUPT_GPIO1 at (94.1, 24.0)
- removed the INTERRUPT_GPIO1 at (231.3, 26.6)
- removed the INTERRUPT_GPIO1 at (163.7, 177.7)
- removed the INTERRUPT_GPIO1 at (160.1, 24.0)
- removed the R1 at (35.4, 158.3)
- removed the R1 at (250.6, 35.4)
- removed the R1 at (113.5, 32.8)
- removed the R1 at (172.5, 158.3)
- removed the R1 at (179.5, 32.8)
- removed the R2 at (229.9, 146.7)
- removed the R2 at (92.8, 146.7)
- removed the R2 at (262.2, 92.8)
- removed the R2 at (191.1, 90.2)
- removed the R2 at (125.1, 90.2)
- removed the REF** at (155.2, 23.6)
- removed the REF** at (128.9, 120.3)
- removed the REF** at (226.3, 26.2)
- removed the REF** at (26.3, 143.0)
- removed the REF** at (265.9, 26.3)
- removed the REF** at (194.8, 23.8)
- removed the REF** at (155.1, 120.4)
- removed the REF** at (163.5, 143.0)
- removed the REF** at (163.3, 182.6)
- removed the REF** at (194.9, 120.3)
- removed the REF** at (260.0, 142.9)
- removed the REF** at (122.9, 182.8)
- removed the REF** at (266.0, 122.8)
- removed the REF** at (128.7, 23.8)
- removed the REF** at (226.2, 122.9)
- removed the REF** at (26.2, 182.6)
- removed the REF** at (89.1, 23.6)
- removed the REF** at (122.8, 142.9)
- removed the REF** at (260.1, 182.8)
- removed the REF** at (89.0, 120.4)
- removed the SCL1 at (177.3, 38.7)
- removed the SCL1 at (248.4, 41.2)
- removed the SCL1 at (178.4, 160.5)
- removed the SCL1 at (41.2, 160.5)
- removed the SCL1 at (111.2, 38.7)
- removed the SDA1 at (41.2, 154.0)
- removed the SDA1 at (254.9, 41.2)
- removed the SDA1 at (183.8, 38.7)
- removed the SDA1 at (178.4, 154.0)
- removed the SDA1 at (117.7, 38.7)
- removed the SIGNAL_IN1 at (163.8, 149.1)
- removed the SIGNAL_IN1 at (259.8, 26.7)
- removed the SIGNAL_IN1 at (122.6, 24.1)
- removed the SIGNAL_IN1 at (26.7, 149.1)
- removed the SIGNAL_IN1 at (188.7, 24.1)
- removed the U1 at (173.9, 85.7)
- removed the U1 at (245.1, 88.3)
- removed the U1 at (88.3, 163.9)
- removed the U1 at (225.4, 163.9)
- removed the U1 at (107.9, 85.7)
- removed the VCC1 at (104.7, 38.7)
- removed the VCC1 at (241.9, 41.2)
- removed the VCC1 at (178.4, 167.1)
- removed the VCC1 at (41.2, 167.1)
- removed the VCC1 at (170.7, 38.7)
- added 100nF1: CAP, Capacitor_THT:C_Disc_D4.3mm_W1.9mm_P5.00mm, F.Cu at (35.7, 153.9)
- added 100nF1: CAP, Capacitor_THT:C_Disc_D4.3mm_W1.9mm_P5.00mm, F.Cu at (72.2, 30.6)
- added 100nF1: CAP, Capacitor_THT:C_Disc_D4.3mm_W1.9mm_P5.00mm, F.Cu at (170.3, 156.4)
- added 100nF1: CAP, Capacitor_THT:C_Disc_D4.3mm_W1.9mm_P5.00mm, F.Cu at (234.8, 30.6)
- added 100nF1: CAP, Capacitor_THT:C_Disc_D4.3mm_W1.9mm_P5.00mm, F.Cu at (181.4, 30.6)
- added 100nF1: CAP, Capacitor_THT:C_Disc_D4.3mm_W1.9mm_P5.00mm, F.Cu at (123.0, 30.6)
- added 3V3_OUT1: TestPoint, TestPoint:TestPoint_Keystone_5015_Micro-Minature, B.Cu at (88.9, 21.8)
- added 3V3_OUT1: TestPoint, TestPoint:TestPoint_Keystone_5015_Micro-Minature, B.Cu at (198.1, 21.8)
- added 3V3_OUT1: TestPoint, TestPoint:TestPoint_Keystone_5015_Micro-Minature, B.Cu at (161.5, 139.7)
- added 3V3_OUT1: TestPoint, TestPoint:TestPoint_Keystone_5015_Micro-Minature, B.Cu at (251.5, 21.8)
- added 3V3_OUT1: TestPoint, TestPoint:TestPoint_Keystone_5015_Micro-Minature, B.Cu at (139.7, 21.8)
- added 3V3_OUT1: TestPoint, TestPoint:TestPoint_Keystone_5015_Micro-Minature, B.Cu at (26.9, 137.1)
- added BATTERY1: Battery_Cell, Connector_Wire:SolderWire-0.1sqmm_1x02_P3.6mm_D0.4mm_OD1mm, B.Cu at (26.9, 151.3)
- added BATTERY1: Battery_Cell, Connector_Wire:SolderWire-0.1sqmm_1x02_P3.6mm_D0.4mm_OD1mm, B.Cu at (237.3, 21.8)
- added BATTERY1: Battery_Cell, Connector_Wire:SolderWire-0.1sqmm_1x02_P3.6mm_D0.4mm_OD1mm, B.Cu at (183.9, 21.8)
- added BATTERY1: Battery_Cell, Connector_Wire:SolderWire-0.1sqmm_1x02_P3.6mm_D0.4mm_OD1mm, B.Cu at (125.5, 21.8)
- added BATTERY1: Battery_Cell, Connector_Wire:SolderWire-0.1sqmm_1x02_P3.6mm_D0.4mm_OD1mm, B.Cu at (74.7, 21.8)
- added BATTERY1: Battery_Cell, Connector_Wire:SolderWire-0.1sqmm_1x02_P3.6mm_D0.4mm_OD1mm, B.Cu at (161.5, 153.9)
- added BZ1: Buzzer, Buzzer_Beeper:MagneticBuzzer_ProSignal_ABI-009-RC, F.Cu at (148.7, 32.9)
- added BZ1: Buzzer, Buzzer_Beeper:MagneticBuzzer_ProSignal_ABI-009-RC, F.Cu at (172.6, 130.7)
- added BZ1: Buzzer, Buzzer_Beeper:MagneticBuzzer_ProSignal_ABI-009-RC, F.Cu at (207.1, 32.9)
- added BZ1: Buzzer, Buzzer_Beeper:MagneticBuzzer_ProSignal_ABI-009-RC, F.Cu at (260.5, 32.9)
- added BZ1: Buzzer, Buzzer_Beeper:MagneticBuzzer_ProSignal_ABI-009-RC, F.Cu at (97.9, 32.9)
- added BZ1: Buzzer, Buzzer_Beeper:MagneticBuzzer_ProSignal_ABI-009-RC, F.Cu at (38.0, 128.2)
- added D1: EMITTER, LED_THT:LED_D3.0mm_Clear, F.Cu at (253.2, 145.1)
- added D1: EMITTER, LED_THT:LED_D3.0mm_Clear, F.Cu at (83.5, 113.5)
- added D1: EMITTER, LED_THT:LED_D3.0mm_Clear, F.Cu at (192.7, 113.5)
- added D1: EMITTER, LED_THT:LED_D3.0mm_Clear, F.Cu at (246.1, 113.5)
- added D1: EMITTER, LED_THT:LED_D3.0mm_Clear, F.Cu at (118.5, 142.5)
- added D1: EMITTER, LED_THT:LED_D3.0mm_Clear, F.Cu at (134.3, 113.5)
- added GND1: TestPoint, TestPoint:TestPoint_Pad_2.0x2.0mm, B.Cu at (238.1, 42.0)
- added GND1: TestPoint, TestPoint:TestPoint_Pad_2.0x2.0mm, B.Cu at (126.4, 42.0)
- added GND1: TestPoint, TestPoint:TestPoint_Pad_2.0x2.0mm, B.Cu at (47.1, 150.5)
- added GND1: TestPoint, TestPoint:TestPoint_Pad_2.0x2.0mm, B.Cu at (75.6, 42.0)
- added GND1: TestPoint, TestPoint:TestPoint_Pad_2.0x2.0mm, B.Cu at (181.7, 153.0)
- added GND1: TestPoint, TestPoint:TestPoint_Pad_2.0x2.0mm, B.Cu at (184.8, 42.0)
- added INTERRUPT_GPIO1: SW_Push, Connector_Wire:SolderWire-0.1sqmm_1x02_P3.6mm_D0.4mm_OD1mm, B.Cu at (161.5, 130.0)
- added INTERRUPT_GPIO1: SW_Push, Connector_Wire:SolderWire-0.1sqmm_1x02_P3.6mm_D0.4mm_OD1mm, B.Cu at (149.4, 21.8)
- added INTERRUPT_GPIO1: SW_Push, Connector_Wire:SolderWire-0.1sqmm_1x02_P3.6mm_D0.4mm_OD1mm, B.Cu at (98.6, 21.8)
- added INTERRUPT_GPIO1: SW_Push, Connector_Wire:SolderWire-0.1sqmm_1x02_P3.6mm_D0.4mm_OD1mm, B.Cu at (261.2, 21.8)
- added INTERRUPT_GPIO1: SW_Push, Connector_Wire:SolderWire-0.1sqmm_1x02_P3.6mm_D0.4mm_OD1mm, B.Cu at (26.9, 127.4)
- added INTERRUPT_GPIO1: SW_Push, Connector_Wire:SolderWire-0.1sqmm_1x02_P3.6mm_D0.4mm_OD1mm, B.Cu at (207.8, 21.8)
- added R1: 120, Resistor_THT:R_Axial_DIN0204_L3.6mm_D1.6mm_P7.62mm_Horizontal, F.Cu at (82.6, 35.7)
- added R1: 120, Resistor_THT:R_Axial_DIN0204_L3.6mm_D1.6mm_P7.62mm_Horizontal, F.Cu at (133.4, 35.7)
- added R1: 120, Resistor_THT:R_Axial_DIN0204_L3.6mm_D1.6mm_P7.62mm_Horizontal, F.Cu at (175.4, 146.0)
- added R1: 120, Resistor_THT:R_Axial_DIN0204_L3.6mm_D1.6mm_P7.62mm_Horizontal, F.Cu at (191.8, 35.7)
- added R1: 120, Resistor_THT:R_Axial_DIN0204_L3.6mm_D1.6mm_P7.62mm_Horizontal, F.Cu at (40.8, 143.5)
- added R1: 120, Resistor_THT:R_Axial_DIN0204_L3.6mm_D1.6mm_P7.62mm_Horizontal, F.Cu at (245.1, 35.7)
- added R2: 120, Resistor_THT:R_Axial_DIN0204_L3.6mm_D1.6mm_P7.62mm_Horizontal, F.Cu at (77.8, 35.7)
- added R2: 120, Resistor_THT:R_Axial_DIN0204_L3.6mm_D1.6mm_P7.62mm_Horizontal, F.Cu at (187.1, 35.7)
- added R2: 120, Resistor_THT:R_Axial_DIN0204_L3.6mm_D1.6mm_P7.62mm_Horizontal, F.Cu at (40.8, 148.2)
- added R2: 120, Resistor_THT:R_Axial_DIN0204_L3.6mm_D1.6mm_P7.62mm_Horizontal, F.Cu at (128.6, 35.7)
- added R2: 120, Resistor_THT:R_Axial_DIN0204_L3.6mm_D1.6mm_P7.62mm_Horizontal, F.Cu at (240.4, 35.7)
- added R2: 120, Resistor_THT:R_Axial_DIN0204_L3.6mm_D1.6mm_P7.62mm_Horizontal, F.Cu at (175.4, 150.8)
- added REF**: MountingHole_2.2mm_M2, MountingHole:MountingHole_2.2mm_M2, F.Cu at (22.8, 154.8)
- added REF**: MountingHole_2.2mm_M2, MountingHole:MountingHole_2.2mm_M2, F.Cu at (71.3, 114.5)
- added REF**: MountingHole_2.2mm_M2, MountingHole:MountingHole_2.2mm_M2, F.Cu at (157.4, 157.3)
- added REF**: MountingHole_2.2mm_M2, MountingHole:MountingHole_2.2mm_M2, F.Cu at (261.6, 17.7)
- added REF**: MountingHole_2.2mm_M2, MountingHole:MountingHole_2.2mm_M2, F.Cu at (254.2, 157.3)
- added REF**: MountingHole_2.2mm_M2, MountingHole:MountingHole_2.2mm_M2, F.Cu at (122.1, 17.7)
- added REF**: MountingHole_2.2mm_M2, MountingHole:MountingHole_2.2mm_M2, F.Cu at (122.1, 114.5)
- added REF**: MountingHole_2.2mm_M2, MountingHole:MountingHole_2.2mm_M2, F.Cu at (207.8, 114.5)
- added REF**: MountingHole_2.2mm_M2, MountingHole:MountingHole_2.2mm_M2, F.Cu at (149.4, 114.5)
- added REF**: MountingHole_2.2mm_M2, MountingHole:MountingHole_2.2mm_M2, F.Cu at (149.8, 17.7)
- added REF**: MountingHole_2.2mm_M2, MountingHole:MountingHole_2.2mm_M2, F.Cu at (233.8, 17.7)
- added REF**: MountingHole_2.2mm_M2, MountingHole:MountingHole_2.2mm_M2, F.Cu at (261.2, 114.5)
- added REF**: MountingHole_2.2mm_M2, MountingHole:MountingHole_2.2mm_M2, F.Cu at (254.2, 130.0)
- added REF**: MountingHole_2.2mm_M2, MountingHole:MountingHole_2.2mm_M2, F.Cu at (98.6, 114.5)
- added REF**: MountingHole_2.2mm_M2, MountingHole:MountingHole_2.2mm_M2, F.Cu at (157.4, 129.6)
- added REF**: MountingHole_2.2mm_M2, MountingHole:MountingHole_2.2mm_M2, F.Cu at (119.6, 154.8)
- added REF**: MountingHole_2.2mm_M2, MountingHole:MountingHole_2.2mm_M2, F.Cu at (180.5, 17.7)
- added REF**: MountingHole_2.2mm_M2, MountingHole:MountingHole_2.2mm_M2, F.Cu at (99.0, 17.7)
- added REF**: MountingHole_2.2mm_M2, MountingHole:MountingHole_2.2mm_M2, F.Cu at (71.3, 17.7)
- added REF**: MountingHole_2.2mm_M2, MountingHole:MountingHole_2.2mm_M2, F.Cu at (180.5, 114.5)
- added REF**: MountingHole_2.2mm_M2, MountingHole:MountingHole_2.2mm_M2, F.Cu at (119.6, 127.5)
- added REF**: MountingHole_2.2mm_M2, MountingHole:MountingHole_2.2mm_M2, F.Cu at (22.8, 127.1)
- added REF**: MountingHole_2.2mm_M2, MountingHole:MountingHole_2.2mm_M2, F.Cu at (233.8, 114.5)
- added REF**: MountingHole_2.2mm_M2, MountingHole:MountingHole_2.2mm_M2, F.Cu at (208.2, 17.7)
- added SCL1: TestPoint, TestPoint:TestPoint_Pad_2.0x2.0mm, B.Cu at (92.4, 42.0)
- added SCL1: TestPoint, TestPoint:TestPoint_Pad_2.0x2.0mm, B.Cu at (47.1, 133.7)
- added SCL1: TestPoint, TestPoint:TestPoint_Pad_2.0x2.0mm, B.Cu at (201.6, 42.0)
- added SCL1: TestPoint, TestPoint:TestPoint_Pad_2.0x2.0mm, B.Cu at (181.7, 136.2)
- added SCL1: TestPoint, TestPoint:TestPoint_Pad_2.0x2.0mm, B.Cu at (254.9, 42.0)
- added SCL1: TestPoint, TestPoint:TestPoint_Pad_2.0x2.0mm, B.Cu at (143.2, 42.0)
- added SDA1: TestPoint, TestPoint:TestPoint_Pad_2.0x2.0mm, B.Cu at (196.0, 42.0)
- added SDA1: TestPoint, TestPoint:TestPoint_Pad_2.0x2.0mm, B.Cu at (137.6, 42.0)
- added SDA1: TestPoint, TestPoint:TestPoint_Pad_2.0x2.0mm, B.Cu at (86.8, 42.0)
- added SDA1: TestPoint, TestPoint:TestPoint_Pad_2.0x2.0mm, B.Cu at (47.1, 139.3)
- added SDA1: TestPoint, TestPoint:TestPoint_Pad_2.0x2.0mm, B.Cu at (249.3, 42.0)
- added SDA1: TestPoint, TestPoint:TestPoint_Pad_2.0x2.0mm, B.Cu at (181.7, 141.8)
- added SIGNAL_IN1: TestPoint, TestPoint:TestPoint_Keystone_5015_Micro-Minature, B.Cu at (81.1, 21.8)
- added SIGNAL_IN1: TestPoint, TestPoint:TestPoint_Keystone_5015_Micro-Minature, B.Cu at (161.5, 147.5)
- added SIGNAL_IN1: TestPoint, TestPoint:TestPoint_Keystone_5015_Micro-Minature, B.Cu at (26.9, 144.9)
- added SIGNAL_IN1: TestPoint, TestPoint:TestPoint_Keystone_5015_Micro-Minature, B.Cu at (131.9, 21.8)
- added SIGNAL_IN1: TestPoint, TestPoint:TestPoint_Keystone_5015_Micro-Minature, B.Cu at (190.3, 21.8)
- added SIGNAL_IN1: TestPoint, TestPoint:TestPoint_Keystone_5015_Micro-Minature, B.Cu at (243.7, 21.8)
- added U1: ESP32_DevKit_V1_DOIT, esp32_devkit_v1_doit:esp32_devkit_v1_doit, F.Cu at (246.6, 86.0)
- added U1: ESP32_DevKit_V1_DOIT, esp32_devkit_v1_doit:esp32_devkit_v1_doit, F.Cu at (134.8, 86.0)
- added U1: ESP32_DevKit_V1_DOIT, esp32_devkit_v1_doit:esp32_devkit_v1_doit, F.Cu at (91.0, 142.1)
- added U1: ESP32_DevKit_V1_DOIT, esp32_devkit_v1_doit:esp32_devkit_v1_doit, F.Cu at (193.2, 86.0)
- added U1: ESP32_DevKit_V1_DOIT, esp32_devkit_v1_doit:esp32_devkit_v1_doit, F.Cu at (225.7, 144.6)
- added U1: ESP32_DevKit_V1_DOIT, esp32_devkit_v1_doit:esp32_devkit_v1_doit, F.Cu at (84.0, 86.0)
- added VCC1: TestPoint, TestPoint:TestPoint_Pad_2.0x2.0mm, B.Cu at (243.8, 42.0)
- added VCC1: TestPoint, TestPoint:TestPoint_Pad_2.0x2.0mm, B.Cu at (190.5, 42.0)
- added VCC1: TestPoint, TestPoint:TestPoint_Pad_2.0x2.0mm, B.Cu at (181.7, 147.3)
- added VCC1: TestPoint, TestPoint:TestPoint_Pad_2.0x2.0mm, B.Cu at (81.3, 42.0)
- added VCC1: TestPoint, TestPoint:TestPoint_Pad_2.0x2.0mm, B.Cu at (47.1, 144.8)
- added VCC1: TestPoint, TestPoint:TestPoint_Pad_2.0x2.0mm, B.Cu at (132.1, 42.0)
- moved REF** 102.7 mm to (23.2, 17.7)
- moved REF** 94.1 mm to (50.5, 114.5)
- moved R2 63.5 mm to (29.8, 35.7)
- moved 100nF1 57.1 mm to (24.1, 30.6)
- moved REF** 43.2 mm to (23.2, 114.5)
- moved SIGNAL_IN1 26.8 mm to (33.1, 21.8)
- moved BATTERY1 25.5 mm to (26.7, 21.8)
- moved BZ1 20.2 mm to (49.8, 32.9), turned to 180 degrees
- moved INTERRUPT_GPIO1 19.5 mm to (50.6, 21.8), turned to 180 degrees
- moved SDA1 16.5 mm to (38.7, 42.0)
- moved R1 16.3 mm to (34.5, 35.7), turned to 90 degrees
- moved REF** 16.1 mm to (50.9, 17.7)
- moved D1 13.4 mm to (35.5, 113.5), turned to 0 degrees
- moved VCC1 9.24 mm to (33.2, 42.0)
- moved U1 9.05 mm to (36.0, 86.0)
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Routing:
- net Net-(D1-Pad1): track 213.0 -> 560.9 mm
- net Net-(100nF1-Pad2): track 28.2 -> 313.1 mm
- net Net-(100nF1-Pad1): track 299.9 -> 88.0 mm
- net Net-(3V3_OUT1-Pad1): track 246.6 -> 342.0 mm
- net Net-(INTERRUPT_GPIO1-Pad1): track 319.2 -> 376.7 mm
- net Net-(BZ1-Pad1): track 234.8 -> 270.9 mm
- net Net-(BATTERY1-Pad1): track 197.6 -> 232.0 mm
- net Net-(D1-Pad2): track 250.0 -> 223.4 mm
- net Net-(BZ1-Pad2): track 73.8 -> 55.2 mm
- net Net-(SCL1-Pad1): track 264.3 -> 249.0 mm
- net Net-(SDA1-Pad1): track 325.7 -> 318.6 mm
Other:
- board size 246.4 x 165.7 mm -> 244.2 x 145.5 mm
