File: receptor_circuit/glucometer-pcb.kicad_pcb (KiCad board)
At the start: 2 copper layers, 236.6 x 148.2 mm, 210 parts

Commit message: Agrandamos los pads
Parts:
- removed C25, C28: 15p, Capacitor_THT:C_Disc_D4.3mm_W1.9mm_P5.00mm
- removed C26, C29: 100n, Capacitor_THT:C_Disc_D4.3mm_W1.9mm_P5.00mm
- removed C27, C30: 10u, Capacitor_THT:C_Disc_D4.3mm_W1.9mm_P5.00mm
- removed GND10, GND9, VCC10, VCC9: TestPoint, TestPoint:TestPoint_Keystone_5015_Micro-Minature
- removed LM1458N10, LM1458N9: LM1458N, Custom:MC1458N
- removed R57, R63, R64, R70: 100k, Resistor_THT:R_Axial_DIN0204_L3.6mm_D1.6mm_P7.62mm_Horizontal
- removed R58, R65: 330k, Resistor_THT:R_Axial_DIN0204_L3.6mm_D1.6mm_P7.62mm_Horizontal
- removed R59, R60, R66, R67: 10k, Resistor_THT:R_Axial_DIN0204_L3.6mm_D1.6mm_P7.62mm_Horizontal
- removed R61, R68: 25k, Resistor_THT:R_Axial_DIN0204_L3.6mm_D1.6mm_P7.62mm_Horizontal
- removed R62, R69: 1k, Resistor_THT:R_Axial_DIN0204_L3.6mm_D1.6mm_P7.62mm_Horizontal
- removed RC4558IP17, RC4558IP18, RC4558IP19, RC4558IP20: RC4558IP, Custom:DIP794W53P254L959H508Q8N
- removed RECEPTOR_DIODE10, RECEPTOR_DIODE9: D_Photo, LED_SMD:LED_2512_6332Metric
- removed REF**29, REF**30, REF**31, REF**32, REF**33, REF**34, REF**35, REF**36: MountingHole_2.2mm_M2_ISO7380, MountingHole:MountingHole_2.2mm_M2_ISO7380
- removed S_OUT10, S_OUT9: SIGNAL_OUT, TestPoint:TestPoint_Keystone_5015_Micro-Minature
- moved C13 197.0 mm to (47.2, 142.6)
- moved C14 197.0 mm to (54.6, 113.7)
- moved C15 197.0 mm to (54.7, 117.1)
- moved GND5 197.0 mm to (46.0, 100.2)
- moved LM1458N5 197.0 mm to (42.4, 137.4)
- moved R32 197.0 mm to (41.9, 109.2)
- moved R33 197.0 mm to (59.2, 131.5)
- moved RC4558IP9 197.0 mm to (64.3, 112.5)
- moved RECEPTOR_DIODE5 197.0 mm to (55.5, 157.1)
- moved REF**13 197.0 mm to (70.7, 158.0)
- moved REF**15 197.0 mm to (70.7, 96.0)
- moved REF**16 197.0 mm to (40.4, 95.9)
- moved S_OUT5 197.0 mm to (67.1, 100.2)
- moved R29 197.0 mm to (42.2, 147.5)
- moved R30 197.0 mm to (66.9, 147.3)
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Routing:
- net VCC: track 1149.3 -> 926.2 mm
- net /PWD_1.65: track 1006.4 -> 805.1 mm
- net Net-(R6-Pad1): track 707.6 -> 567.3 mm
- net /SIGNAL_1: track 625.7 -> 497.7 mm
- net Net-(R7-Pad1): track 529.2 -> 423.4 mm
- net Net-(C1-Pad2): track 478.5 -> 382.8 mm
- net Net-(R3-Pad2): track 244.5 -> 192.7 mm
- net Net-(C1-Pad1): track 228.7 -> 183.0 mm
- net /SIGNAL_2: track 173.1 -> 138.5 mm
- net Net-(C3-Pad1): track 117.4 -> 93.9 mm
- net GND: track 31.6 -> 25.2 mm
Other:
- board size 236.6 x 148.2 mm -> 231.6 x 145.8 mm

Commit message: pcb update
Parts:
- removed C10, C13, C16, C19, C22, C4, C7: 15p, Capacitor_THT:C_Disc_D4.3mm_W1.9mm_P5.00mm
- removed C11, C14, C17, C20, C23, C5, C8: 100n, Capacitor_THT:C_Disc_D4.3mm_W1.9mm_P5.00mm
- removed C12, C15, C18, C21, C24, C6, C9: 10u, Capacitor_THT:C_Disc_D4.3mm_W1.9mm_P5.00mm
- removed GND2, GND3, GND4, GND5, GND6, GND7, GND8, VCC2, VCC3, VCC4, VCC5, VCC6, VCC7, VCC8: TestPoint, TestPoint:TestPoint_Keystone_5015_Micro-Minature
- removed LM1458N2, LM1458N3, LM1458N4, LM1458N5, LM1458N6, LM1458N7, LM1458N8: LM1458N, Custom:MC1458N
- removed R10, R11, R17, R18, R24, R25, R31, R32, R38, R39, R45, R46, R52, R53: 10k, Resistor_THT:R_Axial_DIN0204_L3.6mm_D1.6mm_P7.62mm_Horizontal
- removed R12, R19, R26, R33, R40, R47, R54: 25k, Resistor_THT:R_Axial_DIN0204_L3.6mm_D1.6mm_P7.62mm_Horizontal
- removed R13, R20, R27, R34, R41, R48, R55: 1k, Resistor_THT:R_Axial_DIN0204_L3.6mm_D1.6mm_P7.62mm_Horizontal
- removed R14, R15, R21, R22, R28, R29, R35, R36, R42, R43, R49, R50, R56, R8: 100k, Resistor_THT:R_Axial_DIN0204_L3.6mm_D1.6mm_P7.62mm_Horizontal
- removed R16, R23, R30, R37, R44, R51, R9: 330k, Resistor_THT:R_Axial_DIN0204_L3.6mm_D1.6mm_P7.62mm_Horizontal
- removed RC4558IP10, RC4558IP11, RC4558IP12, RC4558IP13, RC4558IP14, RC4558IP15, RC4558IP16, RC4558IP3, RC4558IP4, RC4558IP5, RC4558IP6, RC4558IP7, RC4558IP8, RC4558IP9: RC4558IP, Custom:DIP794W53P254L959H508Q8N
- removed RECEPTOR_DIODE2, RECEPTOR_DIODE3, RECEPTOR_DIODE4, RECEPTOR_DIODE5, RECEPTOR_DIODE6, RECEPTOR_DIODE7, RECEPTOR_DIODE8: D_Photo, LED_SMD:LED_2512_6332Metric
- removed REF**1, REF**10, REF**11, REF**12, REF**13, REF**14, REF**15, REF**16, REF**17, REF**18, REF**19, REF**2, REF**20, REF**21, REF**22, REF**23, REF**24, REF**25, REF**26, REF**27, REF**28, REF**3, REF**4, REF**5, REF**6, REF**7, REF**8, REF**9: MountingHole_2.2mm_M2_ISO7380, MountingHole:MountingHole_2.2mm_M2_ISO7380
- removed S_OUT2, S_OUT3, S_OUT4, S_OUT5, S_OUT6, S_OUT7, S_OUT8: SIGNAL_OUT, TestPoint:TestPoint_Keystone_5015_Micro-Minature
- moved R3 90.1 mm to (115.4, 79.8), turned to -90 degrees
- moved R4 89.7 mm to (112.1, 87.5), turned to 90 degrees
- moved C2 88.2 mm to (114.9, 100.6)
- moved R1 84.7 mm to (123.7, 93.2), turned to -90 degrees
- moved C3 83.2 mm to (111.2, 100.6), turned to 90 degrees
- moved REF** 81.2 mm to (134.6, 68.6)
- moved C1 80.8 mm to (119.7, 100.6), turned to 90 degrees
- moved REF** 78.4 mm to (137.2, 121.9)
- moved LM1458N1 77.9 mm to (107.4, 102.8), turned to -90 degrees
- moved VCC1 77.6 mm to (114.3, 75.1)
- moved GND1 77.1 mm to (102.5, 75.1)
- moved S_OUT1 76.8 mm to (123.1, 75.1)
- moved R5 75.5 mm to (126.8, 87.6), turned to 90 degrees
- moved RECEPTOR_DIODE1 73.4 mm to (113.0, 125.1), turned to 0 degrees
- moved RC4558IP1 73.2 mm to (103.6, 96.8), turned to 90 degrees
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Routing:
- net VCC: track 926.2 -> 91.1 mm
- net /PWD_1.65: track 805.1 -> 47.1 mm
- net Net-(R6-Pad1): track 567.3 -> 35.7 mm
- net /SIGNAL_1: track 497.7 -> 38.8 mm
- net Net-(R7-Pad1): track 423.4 -> 17.1 mm
- net Net-(C1-Pad2): track 382.8 -> 30.3 mm
- net Net-(R3-Pad2): track 192.7 -> 16.7 mm
- net Net-(C1-Pad1): track 183.0 -> 55.3 mm
- net /SIGNAL_2: track 138.5 -> 44.2 mm
- net Net-(C3-Pad1): track 93.9 -> 10.1 mm
- net GND: track 25.2 -> 0.09 mm
Other:
- board size 231.6 x 145.8 mm -> 35.5 x 60.6 mm

Commit message: rework receptor PCB
Parts:
- moved REF** 13.2 mm to (127.9, 131.3)
- moved REF** 12.4 mm to (99.7, 131.3)
- moved REF** 10.9 mm to (99.7, 70.5)
- moved REF** 6.96 mm to (127.9, 70.5)
- moved RECEPTOR_DIODE1 5.53 mm to (113.8, 130.6)
- moved R5 0.93 mm to (125.9, 87.5)
- moved R7 0.89 mm to (118.5, 79.9)
- moved R6 0.89 mm to (122.2, 79.9)
- moved R4 0.68 mm to (111.5, 87.4)
- moved R3 0.48 mm to (115.0, 79.8)
Routing:
- net Net-(C1-Pad1): track 55.3 -> 49.7 mm
- net /PWD_1.65: track 47.1 -> 44.8 mm
- net VCC: track 91.1 -> 88.9 mm
Other:
- board size 35.5 x 60.6 mm -> 33.3 x 65.6 mm

Commit message: rework receptor PCB
Parts:
- moved S_OUT1 9.25 mm to (113.9, 75.1)
- moved VCC1 7.87 mm to (122.2, 75.1)
- moved REF** 3.65 mm to (127.9, 74.1)
- moved REF** 3.63 mm to (99.7, 74.1)
- moved GND1 3.11 mm to (105.6, 75.1)
Routing:
- net VCC: track 88.9 -> 80.7 mm
- net Net-(R6-Pad1): track 35.4 -> 41.8 mm
- net Net-(C1-Pad1): track 49.7 -> 55.1 mm
Other:
- board size 33.3 x 65.6 mm -> 33.3 x 62 mm
Changed lines of the file:
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@@
   )
   (footprint "MountingHole:MountingHole_2.2mm_M2_ISO7380" (layer "F.Cu")
-    (at 99.681023 70.452334)
+    (at 99.65968 74.081997)
     (descr "Mounting Hole 2.2mm, no annular, M2, ISO7380")
     (tags "mounting hole 2.2mm no annular m2 iso7380")
@@
   )
   (footprint "MountingHole:MountingHole_2.2mm_M2_ISO7380" (layer "F.Cu")
-    (at 127.912846 70.452334)
+    (at 127.89199 74.104207)
     (descr "Mounting Hole 2.2mm, no annular, M2, ISO7380")
     (tags "mounting hole 2.2mm no annular m2 iso7380")
@@
   )
   (footprint "TestPoint:TestPoint_Keystone_5015_Micro-Minature" (layer "B.Cu")
-    (at 123.119765 75.053057)
+    (at 113.869295 75.053111)
     (descr "SMT Test Point- Micro Miniature 5015, http://www.keyelco.com/product-pdf.cfm?p=1353")
     (tags "Test Point")
@@
   )
   (footprint "TestPoint:TestPoint_Keystone_5015_Micro-Minature" (layer "B.Cu")
-    (at 114.3 75.053057)
+    (at 122.167368 75.053111)
     (descr "SMT Test Point- Micro Miniature 5015, http://www.keyelco.com/product-pdf.cfm?p=1353")
     (tags "Test Point")
@@
   )
   (footprint "TestPoint:TestPoint_Keystone_5015_Micro-Minature" (layer "B.Cu")
-    (at 102.524667 75.053057)
+    (at 105.638686 75.053111)
     (descr "SMT Test Point- Micro Miniature 5015, http://www.keyelco.com/product-pdf.cfm?p=1353")
     (tags "Test Point")
@@
     )
   )
-  (gr_rect (start 130.484496 133.689187) (end 97.149664 68.055279) (layer "Edge.Cuts") (width 0.1) (fill none))
+  (gr_rect (start 130.484496 133.689187) (end 97.149664 71.698337) (layer "Edge.Cuts") (width 0.1) (fill none))
+  (segment (start 108.876264 114.598759) (end 105.271959 114.598759) (width 0.25) (layer "B.Cu") (net 1))
   (segment (start 119.936229 100.801028) (end 119.745211 100.61001) (width 0.25) (layer "B.Cu") (net 1))
+  (segment (start 104.824414 114.151214) (end 104.824414 112.915269) (width 0.25) (layer "B.Cu") (net 1))
+  (segment (start 117.78564 103.890343) (end 117.78564 103.957807) (width 0.25) (layer "B.Cu") (net 1))
   (segment (start 116.705071 130.565598) (end 116.699012 130.571657) (width 0.25) (layer "B.Cu") (net 1))
+  (segment (start 105.271959 114.598759) (end 104.824414 114.151214) (width 0.25) (layer "B.Cu") (net 1))
   (segment (start 123.685277 100.801028) (end 119.936229 100.801028) (width 0.25) (layer "B.Cu") (net 1))
-  (segment (start 104.824414 113.905258) (end 104.824414 112.915269) (width 0.25) (layer "B.Cu") (net 1))
-  (segment (start 116.705071 111.58124) (end 113.687552 114.598759) (width 0.25) (layer "B.Cu") (net 1))
+  (segment (start 109.352639 112.390808) (end 109.352639 114.122384) (width 0.25) (layer "B.Cu") (net 1))
   (segment (start 119.745211 101.960667) (end 116.705071 105.000807) (width 0.25) (layer "B.Cu") (net 1))
   (segment (start 116.705071 105.000807) (end 116.705071 130.565598) (width 0.25) (layer "B.Cu") (net 1))
-  (segment (start 105.517915 114.598759) (end 104.824414 113.905258) (width 0.25) (layer "B.Cu") (net 1))
+  (segment (start 109.352639 114.122384) (end 108.876264 114.598759) (width 0.25) (layer "B.Cu") (net 1))
   (segment (start 119.745211 100.61001) (end 119.745211 101.960667) (width 0.25) (layer "B.Cu") (net 1))
-  (segment (start 113.687552 114.598759) (end 105.517915 114.598759) (width 0.25) (layer "B.Cu") (net 1))
+  (segment (start 117.78564 103.957807) (end 109.352639 112.390808) (width 0.25) (layer "B.Cu") (net 1))
   (segment (start 99.774601 79.804759) (end 105.621005 85.651163) (width 0.25) (layer "B.Cu") (net 2))
   (segment (start 105.621005 85.651163) (end 116.131163 85.651163) (width 0.25) (layer "B.Cu") (net 2))
@@
   (segment (start 114.858891 94.125402) (end 118.272064 90.712229) (width 0.25) (layer "B.Cu") (net 6))
   (segment (start 119.153174 90.712229) (end 122.156124 87.709279) (width 0.25) (layer "B.Cu") (net 6))
-  (segment (start 116.458694 72.894363) (end 114.3 75.053057) (width 0.25) (layer "B.Cu") (net 7))
-  (segment (start 128.565204 75.225204) (end 126.234363 72.894363) (width 0.25) (layer "B.Cu") (net 7))
-  (segment (start 122.521302 90.289653) (end 126.929327 90.289653) (width 0.25) (layer "B.Cu") (net 7))
+  (segment (start 102.223833 98.2618) (end 99.744414 100.741219) (width 0.25) (layer "B.Cu") (net 7))
+  (segment (start 115.554099 98.2618) (end 102.223833 98.2618) (width 0.25) (layer "B.Cu") (net 7))
+  (segment (start 116.84 94.601022) (end 116.84 96.975899) (width 0.25) (layer "B.Cu") (net 7))
+  (segment (start 119.735857 75.053057) (end 124.304817 75.053057) (width 0.25) (layer "B.Cu") (net 7))
   (segment (start 107.394601 79.804759) (end 109.233292 81.64345) (width 0.25) (layer "B.Cu") (net 7))
+  (segment (start 127.742104 83.301631) (end 128.57416 84.133687) (width 0.25) (layer "B.Cu") (net 7))
   (segment (start 99.744414 100.741219) (end 102.24522 103.242025) (width 0.25) (layer "B.Cu") (net 7))
-  (segment (start 120.609046 92.201909) (end 122.521302 90.289653) (width 0.25) (layer "B.Cu") (net 7))
-  (segment (start 116.84 93.98) (end 118.618091 92.201909) (width 0.25) (layer "B.Cu") (net 7))
-  (segment (start 99.744414 100.741219) (end 102.223833 98.2618) (width 0.25) (layer "B.Cu") (net 7))
+  (segment (start 124.304817 75.053057) (end 127.742104 78.490344) (width 0.25) (layer "B.Cu") (net 7))
+  (segment (start 121.151369 90.289653) (end 116.84 94.601022) (width 0.25) (layer "B.Cu") (net 7))
   (segment (start 109.233292 81.64345) (end 113.145464 81.64345) (width 0.25) (layer "B.Cu") (net 7))
-  (segment (start 102.223833 98.2618) (end 115.554099 98.2618) (width 0.25) (layer "B.Cu") (net 7))
-  (segment (start 126.929327 90.289653) (end 128.565204 88.653776) (width 0.25) (layer "B.Cu") (net 7))
-  (segment (start 115.554099 98.2618) (end 116.84 96.975899) (width 0.25) (layer "B.Cu") (net 7))
-  (segment (start 114.971207 79.817707) (end 114.3 79.1465) (width 0.25) (layer "B.Cu") (net 7))
+  (segment (start 127.005747 90.289653) (end 121.151369 90.289653) (width 0.25) (layer "B.Cu") (net 7))
   (segment (start 102.24522 103.242025) (end 105.31117 103.242025) (width 0.25) (layer "B.Cu") (net 7))
-  (segment (start 118.618091 92.201909) (end 120.609046 92.201909) (width 0.25) (layer "B.Cu") (net 7))
   (segment (start 113.145464 81.64345) (end 114.971207 79.817707) (width 0.25) (layer "B.Cu") (net 7))
-  (segment (start 128.565204 88.653776) (end 128.565204 75.225204) (width 0.25) (layer "B.Cu") (net 7))
-  (segment (start 114.3 79.1465) (end 114.3 75.053057) (width 0.25) (layer "B.Cu") (net 7))
+  (segment (start 116.84 96.975899) (end 115.554099 98.2618) (width 0.25) (layer "B.Cu") (net 7))
   (segment (start 105.31117 103.242025) (end 107.364414 105.295269) (width 0.25) (layer "B.Cu") (net 7))
+  (segment (start 128.57416 88.72124) (end 127.005747 90.289653) (width 0.25) (layer "B.Cu") (net 7))
+  (segment (start 127.742104 78.490344) (end 127.742104 83.301631) (width 0.25) (layer "B.Cu") (net 7))
+  (segment (start 128.57416 84.133687) (end 128.57416 88.72124) (width 0.25) (layer "B.Cu") (net 7))
   (segment (start 99.744414 100.741219) (end 99.744414 100.897413) (width 0.25) (layer "B.Cu") (net 7))
-  (segment (start 126.234363 72.894363) (end 116.458694 72.894363) (width 0.25) (layer "B.Cu") (net 7))
-  (segment (start 116.84 96.975899) (end 116.84 93.98) (width 0.25) (layer "B.Cu") (net 7))
+  (segment (start 114.971207 79.817707) (end 119.735857 75.053057) (width 0.25) (layer "B.Cu") (net 7))
   (segment (start 102.284414 105.814403) (end 102.212278 105.814403) (width 0.25) (layer "B.Cu") (net 10))
   (segment (start 102.212278 105.814403) (end 102.212278 105.879148) (width 0.25) (layer "B.Cu") (net 10))
@@
   (segment (start 108.628741 94.790502) (end 106.813697 94.790502) (width 0.25) (layer "B.Cu") (net 12))
   (segment (start 114.947233 87.461681) (end 111.487052 87.461681) (width 0.25) (layer "B.Cu") (net 12))
-  (segment (start 123.041277 78.732474) (end 123.041277 75.131545) (width 0.25) (layer "B.Cu") (net 13))
+  (segment (start 112.992262 75.053111) (end 110.878391 75.053111) (width 0.25) (layer "B.Cu") (net 13))
   (segment (start 118.513067 84.374434) (end 118.513067 87.471439) (width 0.25) (layer "B.Cu") (net 13))
-  (segment (start 123.041277 75.131545) (end 123.119765 75.053057) (width 0.25) (layer "B.Cu") (net 13))
-  (segment (start 121.92 79.853751) (end 123.041277 78.732474) (width 0.25) (layer "B.Cu") (net 13))
+  (segment (start 108.17983 77.751672) (end 104.042037 77.751672) (width 0.25) (layer "B.Cu") (net 13))
   (segment (start 121.92 79.853751) (end 121.92 80.967501) (width 0.25) (layer "B.Cu") (net 13))
+  (segment (start 104.042037 77.751672) (end 102.314601 79.479108) (width 0.25) (layer "B.Cu") (net 13))
   (segment (start 102.314601 79.804759) (end 106.822847 84.313005) (width 0.25) (layer "B.Cu") (net 13))
   (segment (start 116.252425 84.313005) (end 118.513067 86.573647) (width 0.25) (layer "B.Cu") (net 13))
-  (segment (start 123.119765 75.053057) (end 124.249486 75.053057) (width 0.3) (layer "B.Cu") (net 13))
+  (segment (start 110.878391 75.053111) (end 108.17983 77.751672) (width 0.25) (layer "B.Cu") (net 13))
+  (segment (start 112.969774 75.030623) (end 112.992262 75.053111) (width 0.25) (layer "B.Cu") (net 13))
   (segment (start 121.92 80.967501) (end 118.513067 84.374434) (width 0.25) (layer "B.Cu") (net 13))
   (segment (start 106.822847 84.313005) (end 116.252425 84.313005) (width 0.25) (layer "B.Cu") (net 13))
+  (segment (start 102.314601 79.479108) (end 102.314601 79.804759) (width 0.25) (layer "B.Cu") (net 13))
   (segment (start 118.513067 86.573647) (end 118.513067 87.471439) (width 0.25) (layer "B.Cu") (net 13))
   (segment (start 104.854601 79.804759) (end 107.95426 82.904418) (width 0.25) (layer "B.Cu") (net 14))
@@
     (polygon
       (pts
-        (xy 130.455987 68.067794)
+        (xy 130.454636 71.702207)
         (xy 130.445582 133.665897)
         (xy 97.175557 133.664615)
-        (xy 97.123358 68.055404)
+        (xy 97.122007 71.689817)
       )
     )

Commit message: emmiter update
Parts:
- added C1: 15p, Capacitor_THT:C_Disc_D4.3mm_W1.9mm_P5.00mm, F.Cu at (40.3, 137.0)
- added C1: 15p, Capacitor_THT:C_Disc_D4.3mm_W1.9mm_P5.00mm, F.Cu at (85.8, 43.6)
- added C1: 15p, Capacitor_THT:C_Disc_D4.3mm_W1.9mm_P5.00mm, F.Cu at (84.8, 137.2)
- added C1: 15p, Capacitor_THT:C_Disc_D4.3mm_W1.9mm_P5.00mm, F.Cu at (173.2, 138.0)
- added C1: 15p, Capacitor_THT:C_Disc_D4.3mm_W1.9mm_P5.00mm, F.Cu at (216.4, 44.0)
- added C1: 15p, Capacitor_THT:C_Disc_D4.3mm_W1.9mm_P5.00mm, F.Cu at (264.5, 137.5)
- added C1: 15p, Capacitor_THT:C_Disc_D4.3mm_W1.9mm_P5.00mm, F.Cu at (129.8, 137.1)
- added C1: 15p, Capacitor_THT:C_Disc_D4.3mm_W1.9mm_P5.00mm, F.Cu at (263.6, 44.1)
- added C1: 15p, Capacitor_THT:C_Disc_D4.3mm_W1.9mm_P5.00mm, F.Cu at (173.2, 44.1)
- added C1: 15p, Capacitor_THT:C_Disc_D4.3mm_W1.9mm_P5.00mm, F.Cu at (129.0, 43.6)
- added C1: 15p, Capacitor_THT:C_Disc_D4.3mm_W1.9mm_P5.00mm, F.Cu at (216.2, 137.5)
- added C2: 100n, Capacitor_THT:C_Disc_D4.3mm_W1.9mm_P5.00mm, F.Cu at (258.7, 44.1)
- added C2: 100n, Capacitor_THT:C_Disc_D4.3mm_W1.9mm_P5.00mm, F.Cu at (168.3, 138.0)
- added C2: 100n, Capacitor_THT:C_Disc_D4.3mm_W1.9mm_P5.00mm, F.Cu at (211.3, 137.5)
- added C2: 100n, Capacitor_THT:C_Disc_D4.3mm_W1.9mm_P5.00mm, F.Cu at (124.1, 43.6)
- added C2: 100n, Capacitor_THT:C_Disc_D4.3mm_W1.9mm_P5.00mm, F.Cu at (211.5, 44.0)
- added C2: 100n, Capacitor_THT:C_Disc_D4.3mm_W1.9mm_P5.00mm, F.Cu at (35.4, 137.0)
- added C2: 100n, Capacitor_THT:C_Disc_D4.3mm_W1.9mm_P5.00mm, F.Cu at (168.3, 44.1)
- added C2: 100n, Capacitor_THT:C_Disc_D4.3mm_W1.9mm_P5.00mm, F.Cu at (124.9, 137.1)
- added C2: 100n, Capacitor_THT:C_Disc_D4.3mm_W1.9mm_P5.00mm, F.Cu at (259.6, 137.5)
- added C2: 100n, Capacitor_THT:C_Disc_D4.3mm_W1.9mm_P5.00mm, F.Cu at (80.9, 43.6)
- added C2: 100n, Capacitor_THT:C_Disc_D4.3mm_W1.9mm_P5.00mm, F.Cu at (80.0, 137.2)
- added C3: 10u, Capacitor_THT:C_Disc_D4.3mm_W1.9mm_P5.00mm, F.Cu at (207.9, 44.0)
- added C3: 10u, Capacitor_THT:C_Disc_D4.3mm_W1.9mm_P5.00mm, F.Cu at (77.3, 43.6)
- added C3: 10u, Capacitor_THT:C_Disc_D4.3mm_W1.9mm_P5.00mm, F.Cu at (31.8, 137.0)
- added C3: 10u, Capacitor_THT:C_Disc_D4.3mm_W1.9mm_P5.00mm, F.Cu at (164.7, 138.0)
- added C3: 10u, Capacitor_THT:C_Disc_D4.3mm_W1.9mm_P5.00mm, F.Cu at (255.9, 137.5)
- added C3: 10u, Capacitor_THT:C_Disc_D4.3mm_W1.9mm_P5.00mm, F.Cu at (121.2, 137.1)
- added C3: 10u, Capacitor_THT:C_Disc_D4.3mm_W1.9mm_P5.00mm, F.Cu at (255.0, 44.1)
- added C3: 10u, Capacitor_THT:C_Disc_D4.3mm_W1.9mm_P5.00mm, F.Cu at (207.6, 137.5)
- added C3: 10u, Capacitor_THT:C_Disc_D4.3mm_W1.9mm_P5.00mm, F.Cu at (76.3, 137.2)
- added C3: 10u, Capacitor_THT:C_Disc_D4.3mm_W1.9mm_P5.00mm, F.Cu at (120.5, 43.6)
- added C3: 10u, Capacitor_THT:C_Disc_D4.3mm_W1.9mm_P5.00mm, F.Cu at (164.7, 44.1)
- added GND1: TestPoint, TestPoint:TestPoint_Keystone_5015_Micro-Minature, B.Cu at (202.3, 18.4)
- added GND1: TestPoint, TestPoint:TestPoint_Keystone_5015_Micro-Minature, B.Cu at (202.1, 112.0)
- added GND1: TestPoint, TestPoint:TestPoint_Keystone_5015_Micro-Minature, B.Cu at (70.7, 111.7)
- added GND1: TestPoint, TestPoint:TestPoint_Keystone_5015_Micro-Minature, B.Cu at (249.5, 18.6)
- added GND1: TestPoint, TestPoint:TestPoint_Keystone_5015_Micro-Minature, B.Cu at (71.7, 18.1)
- added GND1: TestPoint, TestPoint:TestPoint_Keystone_5015_Micro-Minature, B.Cu at (115.7, 111.6)
- added GND1: TestPoint, TestPoint:TestPoint_Keystone_5015_Micro-Minature, B.Cu at (159.1, 112.4)
- added GND1: TestPoint, TestPoint:TestPoint_Keystone_5015_Micro-Minature, B.Cu at (250.3, 112.0)
- added GND1: TestPoint, TestPoint:TestPoint_Keystone_5015_Micro-Minature, B.Cu at (159.1, 18.6)
- added GND1: TestPoint, TestPoint:TestPoint_Keystone_5015_Micro-Minature, B.Cu at (114.9, 18.1)
- added GND1: TestPoint, TestPoint:TestPoint_Keystone_5015_Micro-Minature, B.Cu at (26.2, 111.4)
- added LM1458N1: LM1458N, Custom:MC1458N, F.Cu at (27.9, 139.1)
- added LM1458N1: LM1458N, Custom:MC1458N, F.Cu at (116.6, 45.8)
- added LM1458N1: LM1458N, Custom:MC1458N, F.Cu at (204.0, 46.1)
- added LM1458N1: LM1458N, Custom:MC1458N, F.Cu at (203.8, 139.7)
- added LM1458N1: LM1458N, Custom:MC1458N, F.Cu at (72.5, 139.4)
- added LM1458N1: LM1458N, Custom:MC1458N, F.Cu at (73.4, 45.8)
- added LM1458N1: LM1458N, Custom:MC1458N, F.Cu at (252.1, 139.7)
- added LM1458N1: LM1458N, Custom:MC1458N, F.Cu at (160.8, 46.3)
- added LM1458N1: LM1458N, Custom:MC1458N, F.Cu at (251.2, 46.3)
- added LM1458N1: LM1458N, Custom:MC1458N, F.Cu at (117.4, 139.3)
- added LM1458N1: LM1458N, Custom:MC1458N, F.Cu at (160.8, 140.1)
- added R1: 100k, Resistor_THT:R_Axial_DIN0204_L3.6mm_D1.6mm_P7.62mm_Horizontal, F.Cu at (44.3, 129.5)
- added R1: 100k, Resistor_THT:R_Axial_DIN0204_L3.6mm_D1.6mm_P7.62mm_Horizontal, F.Cu at (220.1, 130.1)
- added R1: 100k, Resistor_THT:R_Axial_DIN0204_L3.6mm_D1.6mm_P7.62mm_Horizontal, F.Cu at (89.8, 36.2)
- added R1: 100k, Resistor_THT:R_Axial_DIN0204_L3.6mm_D1.6mm_P7.62mm_Horizontal, F.Cu at (177.2, 36.7)
- added R1: 100k, Resistor_THT:R_Axial_DIN0204_L3.6mm_D1.6mm_P7.62mm_Horizontal, F.Cu at (132.9, 36.2)
- added R1: 100k, Resistor_THT:R_Axial_DIN0204_L3.6mm_D1.6mm_P7.62mm_Horizontal, F.Cu at (177.2, 130.5)
- added R1: 100k, Resistor_THT:R_Axial_DIN0204_L3.6mm_D1.6mm_P7.62mm_Horizontal, F.Cu at (267.5, 36.7)
- added R1: 100k, Resistor_THT:R_Axial_DIN0204_L3.6mm_D1.6mm_P7.62mm_Horizontal, F.Cu at (220.3, 36.6)
- added R1: 100k, Resistor_THT:R_Axial_DIN0204_L3.6mm_D1.6mm_P7.62mm_Horizontal, F.Cu at (88.8, 129.8)
- added R1: 100k, Resistor_THT:R_Axial_DIN0204_L3.6mm_D1.6mm_P7.62mm_Horizontal, F.Cu at (268.4, 130.1)
- added R1: 100k, Resistor_THT:R_Axial_DIN0204_L3.6mm_D1.6mm_P7.62mm_Horizontal, F.Cu at (133.7, 129.7)
- added R2: 330k, Resistor_THT:R_Axial_DIN0204_L3.6mm_D1.6mm_P7.62mm_Horizontal, F.Cu at (223.3, 44.2)
- added R2: 330k, Resistor_THT:R_Axial_DIN0204_L3.6mm_D1.6mm_P7.62mm_Horizontal, F.Cu at (135.9, 43.8)
- added R2: 330k, Resistor_THT:R_Axial_DIN0204_L3.6mm_D1.6mm_P7.62mm_Horizontal, F.Cu at (47.2, 137.2)
- added R2: 330k, Resistor_THT:R_Axial_DIN0204_L3.6mm_D1.6mm_P7.62mm_Horizontal, F.Cu at (270.4, 44.3)
- added R2: 330k, Resistor_THT:R_Axial_DIN0204_L3.6mm_D1.6mm_P7.62mm_Horizontal, F.Cu at (180.1, 138.2)
- added R2: 330k, Resistor_THT:R_Axial_DIN0204_L3.6mm_D1.6mm_P7.62mm_Horizontal, F.Cu at (180.1, 44.3)
- added R2: 330k, Resistor_THT:R_Axial_DIN0204_L3.6mm_D1.6mm_P7.62mm_Horizontal, F.Cu at (91.7, 137.4)
- added R2: 330k, Resistor_THT:R_Axial_DIN0204_L3.6mm_D1.6mm_P7.62mm_Horizontal, F.Cu at (271.3, 137.7)
- added R2: 330k, Resistor_THT:R_Axial_DIN0204_L3.6mm_D1.6mm_P7.62mm_Horizontal, F.Cu at (136.6, 137.3)
- added R2: 330k, Resistor_THT:R_Axial_DIN0204_L3.6mm_D1.6mm_P7.62mm_Horizontal, F.Cu at (92.7, 43.8)
- added R2: 330k, Resistor_THT:R_Axial_DIN0204_L3.6mm_D1.6mm_P7.62mm_Horizontal, F.Cu at (223.1, 137.7)
- added R3: 10k, Resistor_THT:R_Axial_DIN0204_L3.6mm_D1.6mm_P7.62mm_Horizontal, F.Cu at (168.4, 117.2)
- added R3: 10k, Resistor_THT:R_Axial_DIN0204_L3.6mm_D1.6mm_P7.62mm_Horizontal, F.Cu at (168.4, 23.3)
- added R3: 10k, Resistor_THT:R_Axial_DIN0204_L3.6mm_D1.6mm_P7.62mm_Horizontal, F.Cu at (35.5, 116.2)
- added R3: 10k, Resistor_THT:R_Axial_DIN0204_L3.6mm_D1.6mm_P7.62mm_Horizontal, F.Cu at (125.0, 116.4)
- added R3: 10k, Resistor_THT:R_Axial_DIN0204_L3.6mm_D1.6mm_P7.62mm_Horizontal, F.Cu at (211.4, 116.8)
- added R3: 10k, Resistor_THT:R_Axial_DIN0204_L3.6mm_D1.6mm_P7.62mm_Horizontal, F.Cu at (211.6, 23.2)
- added R3: 10k, Resistor_THT:R_Axial_DIN0204_L3.6mm_D1.6mm_P7.62mm_Horizontal, F.Cu at (258.8, 23.3)
- added R3: 10k, Resistor_THT:R_Axial_DIN0204_L3.6mm_D1.6mm_P7.62mm_Horizontal, F.Cu at (81.0, 22.8)
- added R3: 10k, Resistor_THT:R_Axial_DIN0204_L3.6mm_D1.6mm_P7.62mm_Horizontal, F.Cu at (259.7, 116.8)
- added R3: 10k, Resistor_THT:R_Axial_DIN0204_L3.6mm_D1.6mm_P7.62mm_Horizontal, F.Cu at (80.1, 116.4)
- added R3: 10k, Resistor_THT:R_Axial_DIN0204_L3.6mm_D1.6mm_P7.62mm_Horizontal, F.Cu at (124.2, 22.8)
- added R4: 10k, Resistor_THT:R_Axial_DIN0204_L3.6mm_D1.6mm_P7.62mm_Horizontal, F.Cu at (255.3, 31.0)
- added R4: 10k, Resistor_THT:R_Axial_DIN0204_L3.6mm_D1.6mm_P7.62mm_Horizontal, F.Cu at (208.1, 30.8)
- added R4: 10k, Resistor_THT:R_Axial_DIN0204_L3.6mm_D1.6mm_P7.62mm_Horizontal, F.Cu at (77.5, 30.5)
- added R4: 10k, Resistor_THT:R_Axial_DIN0204_L3.6mm_D1.6mm_P7.62mm_Horizontal, F.Cu at (164.9, 31.0)
- added R4: 10k, Resistor_THT:R_Axial_DIN0204_L3.6mm_D1.6mm_P7.62mm_Horizontal, F.Cu at (32.0, 123.8)
- added R4: 10k, Resistor_THT:R_Axial_DIN0204_L3.6mm_D1.6mm_P7.62mm_Horizontal, F.Cu at (256.2, 124.4)
- added R4: 10k, Resistor_THT:R_Axial_DIN0204_L3.6mm_D1.6mm_P7.62mm_Horizontal, F.Cu at (164.9, 124.8)
- added R4: 10k, Resistor_THT:R_Axial_DIN0204_L3.6mm_D1.6mm_P7.62mm_Horizontal, F.Cu at (121.5, 124.0)
- added R4: 10k, Resistor_THT:R_Axial_DIN0204_L3.6mm_D1.6mm_P7.62mm_Horizontal, F.Cu at (76.6, 124.0)
- added R4: 10k, Resistor_THT:R_Axial_DIN0204_L3.6mm_D1.6mm_P7.62mm_Horizontal, F.Cu at (120.7, 30.5)
- added R4: 10k, Resistor_THT:R_Axial_DIN0204_L3.6mm_D1.6mm_P7.62mm_Horizontal, F.Cu at (207.9, 124.4)
- added R5: 25k, Resistor_THT:R_Axial_DIN0204_L3.6mm_D1.6mm_P7.62mm_Horizontal, F.Cu at (46.4, 123.8)
- added R5: 25k, Resistor_THT:R_Axial_DIN0204_L3.6mm_D1.6mm_P7.62mm_Horizontal, F.Cu at (222.3, 124.4)
- added R5: 25k, Resistor_THT:R_Axial_DIN0204_L3.6mm_D1.6mm_P7.62mm_Horizontal, F.Cu at (179.3, 124.8)
- added R5: 25k, Resistor_THT:R_Axial_DIN0204_L3.6mm_D1.6mm_P7.62mm_Horizontal, F.Cu at (269.7, 31.0)
- added R5: 25k, Resistor_THT:R_Axial_DIN0204_L3.6mm_D1.6mm_P7.62mm_Horizontal, F.Cu at (270.6, 124.4)
- added R5: 25k, Resistor_THT:R_Axial_DIN0204_L3.6mm_D1.6mm_P7.62mm_Horizontal, F.Cu at (222.5, 30.9)
- added R5: 25k, Resistor_THT:R_Axial_DIN0204_L3.6mm_D1.6mm_P7.62mm_Horizontal, F.Cu at (91.9, 30.5)
- added R5: 25k, Resistor_THT:R_Axial_DIN0204_L3.6mm_D1.6mm_P7.62mm_Horizontal, F.Cu at (135.1, 30.5)
- added R5: 25k, Resistor_THT:R_Axial_DIN0204_L3.6mm_D1.6mm_P7.62mm_Horizontal, F.Cu at (179.3, 31.0)
- added R5: 25k, Resistor_THT:R_Axial_DIN0204_L3.6mm_D1.6mm_P7.62mm_Horizontal, F.Cu at (135.9, 124.0)
- added R5: 25k, Resistor_THT:R_Axial_DIN0204_L3.6mm_D1.6mm_P7.62mm_Horizontal, F.Cu at (91.0, 124.1)
- added R6: 1k, Resistor_THT:R_Axial_DIN0204_L3.6mm_D1.6mm_P7.62mm_Horizontal, F.Cu at (218.6, 116.8)
- added R6: 1k, Resistor_THT:R_Axial_DIN0204_L3.6mm_D1.6mm_P7.62mm_Horizontal, F.Cu at (132.2, 116.4)
- added R6: 1k, Resistor_THT:R_Axial_DIN0204_L3.6mm_D1.6mm_P7.62mm_Horizontal, F.Cu at (87.3, 116.5)
- added R6: 1k, Resistor_THT:R_Axial_DIN0204_L3.6mm_D1.6mm_P7.62mm_Horizontal, F.Cu at (266.0, 23.4)
- added R6: 1k, Resistor_THT:R_Axial_DIN0204_L3.6mm_D1.6mm_P7.62mm_Horizontal, F.Cu at (218.8, 23.2)
- added R6: 1k, Resistor_THT:R_Axial_DIN0204_L3.6mm_D1.6mm_P7.62mm_Horizontal, F.Cu at (266.9, 116.8)
- added R6: 1k, Resistor_THT:R_Axial_DIN0204_L3.6mm_D1.6mm_P7.62mm_Horizontal, F.Cu at (175.6, 117.2)
- added R6: 1k, Resistor_THT:R_Axial_DIN0204_L3.6mm_D1.6mm_P7.62mm_Horizontal, F.Cu at (175.6, 23.4)
- added R6: 1k, Resistor_THT:R_Axial_DIN0204_L3.6mm_D1.6mm_P7.62mm_Horizontal, F.Cu at (131.4, 22.9)
- added R6: 1k, Resistor_THT:R_Axial_DIN0204_L3.6mm_D1.6mm_P7.62mm_Horizontal, F.Cu at (88.2, 22.9)
- added R6: 1k, Resistor_THT:R_Axial_DIN0204_L3.6mm_D1.6mm_P7.62mm_Horizontal, F.Cu at (42.7, 116.2)
- added R7: 100k, Resistor_THT:R_Axial_DIN0204_L3.6mm_D1.6mm_P7.62mm_Horizontal, F.Cu at (128.5, 116.4)
- added R7: 100k, Resistor_THT:R_Axial_DIN0204_L3.6mm_D1.6mm_P7.62mm_Horizontal, F.Cu at (262.3, 23.4)
- added R7: 100k, Resistor_THT:R_Axial_DIN0204_L3.6mm_D1.6mm_P7.62mm_Horizontal, F.Cu at (172.0, 117.2)
- added R7: 100k, Resistor_THT:R_Axial_DIN0204_L3.6mm_D1.6mm_P7.62mm_Horizontal, F.Cu at (83.6, 116.5)
- added R7: 100k, Resistor_THT:R_Axial_DIN0204_L3.6mm_D1.6mm_P7.62mm_Horizontal, F.Cu at (263.2, 116.8)
- added R7: 100k, Resistor_THT:R_Axial_DIN0204_L3.6mm_D1.6mm_P7.62mm_Horizontal, F.Cu at (84.6, 22.9)
- added R7: 100k, Resistor_THT:R_Axial_DIN0204_L3.6mm_D1.6mm_P7.62mm_Horizontal, F.Cu at (39.1, 116.2)
- added R7: 100k, Resistor_THT:R_Axial_DIN0204_L3.6mm_D1.6mm_P7.62mm_Horizontal, F.Cu at (215.2, 23.2)
- added R7: 100k, Resistor_THT:R_Axial_DIN0204_L3.6mm_D1.6mm_P7.62mm_Horizontal, F.Cu at (172.0, 23.4)
- added R7: 100k, Resistor_THT:R_Axial_DIN0204_L3.6mm_D1.6mm_P7.62mm_Horizontal, F.Cu at (127.8, 22.9)
- added R7: 100k, Resistor_THT:R_Axial_DIN0204_L3.6mm_D1.6mm_P7.62mm_Horizontal, F.Cu at (215.0, 116.8)
- added RC4558IP1: RC4558IP, Custom:DIP794W53P254L959H508Q8N, F.Cu at (247.4, 40.3)
- added RC4558IP1: RC4558IP, Custom:DIP794W53P254L959H508Q8N, F.Cu at (200.2, 40.2)
- added RC4558IP1: RC4558IP, Custom:DIP794W53P254L959H508Q8N, F.Cu at (248.3, 133.7)
- added RC4558IP1: RC4558IP, Custom:DIP794W53P254L959H508Q8N, F.Cu at (200.0, 133.7)
- added RC4558IP1: RC4558IP, Custom:DIP794W53P254L959H508Q8N, F.Cu at (68.7, 133.4)
- added RC4558IP1: RC4558IP, Custom:DIP794W53P254L959H508Q8N, F.Cu at (69.6, 39.8)
- added RC4558IP1: RC4558IP, Custom:DIP794W53P254L959H508Q8N, F.Cu at (24.1, 133.1)
- added RC4558IP1: RC4558IP, Custom:DIP794W53P254L959H508Q8N, F.Cu at (113.6, 133.3)
- added RC4558IP1: RC4558IP, Custom:DIP794W53P254L959H508Q8N, F.Cu at (112.8, 39.8)
- added RC4558IP1: RC4558IP, Custom:DIP794W53P254L959H508Q8N, F.Cu at (157.0, 40.3)
- added RC4558IP1: RC4558IP, Custom:DIP794W53P254L959H508Q8N, F.Cu at (157.0, 134.1)
- added RC4558IP2: RC4558IP, Custom:DIP794W53P254L959H508Q8N, F.Cu at (200.2, 27.2)
- added RC4558IP2: RC4558IP, Custom:DIP794W53P254L959H508Q8N, F.Cu at (248.3, 120.7)
- added RC4558IP2: RC4558IP, Custom:DIP794W53P254L959H508Q8N, F.Cu at (112.8, 26.8)
- added RC4558IP2: RC4558IP, Custom:DIP794W53P254L959H508Q8N, F.Cu at (157.1, 121.1)
- added RC4558IP2: RC4558IP, Custom:DIP794W53P254L959H508Q8N, F.Cu at (68.7, 120.4)
- added RC4558IP2: RC4558IP, Custom:DIP794W53P254L959H508Q8N, F.Cu at (69.7, 26.8)
- added RC4558IP2: RC4558IP, Custom:DIP794W53P254L959H508Q8N, F.Cu at (247.4, 27.3)
- added RC4558IP2: RC4558IP, Custom:DIP794W53P254L959H508Q8N, F.Cu at (24.2, 120.1)
- added RC4558IP2: RC4558IP, Custom:DIP794W53P254L959H508Q8N, F.Cu at (113.6, 120.3)
- added RC4558IP2: RC4558IP, Custom:DIP794W53P254L959H508Q8N, F.Cu at (157.1, 27.3)
- added RC4558IP2: RC4558IP, Custom:DIP794W53P254L959H508Q8N, F.Cu at (200.0, 120.7)
- added RECEPTOR_DIODE1: D_Photo, LED_SMD:LED_2512_6332Metric, B.Cu at (123.9, 171.8)
- added RECEPTOR_DIODE1: D_Photo, LED_SMD:LED_2512_6332Metric, B.Cu at (34.4, 171.6)
- added RECEPTOR_DIODE1: D_Photo, LED_SMD:LED_2512_6332Metric, B.Cu at (210.5, 78.6)
- added RECEPTOR_DIODE1: D_Photo, LED_SMD:LED_2512_6332Metric, B.Cu at (210.3, 172.2)
- added RECEPTOR_DIODE1: D_Photo, LED_SMD:LED_2512_6332Metric, B.Cu at (78.9, 171.9)
- added RECEPTOR_DIODE1: D_Photo, LED_SMD:LED_2512_6332Metric, B.Cu at (167.3, 172.6)
- added RECEPTOR_DIODE1: D_Photo, LED_SMD:LED_2512_6332Metric, B.Cu at (123.1, 78.3)
- added RECEPTOR_DIODE1: D_Photo, LED_SMD:LED_2512_6332Metric, B.Cu at (257.6, 78.8)
- added RECEPTOR_DIODE1: D_Photo, LED_SMD:LED_2512_6332Metric, B.Cu at (258.5, 172.2)
- added RECEPTOR_DIODE1: D_Photo, LED_SMD:LED_2512_6332Metric, B.Cu at (79.9, 78.3)
- added RECEPTOR_DIODE1: D_Photo, LED_SMD:LED_2512_6332Metric, B.Cu at (167.3, 78.8)
- added REF**: MountingHole_2.2mm_M2_ISO7380, MountingHole:MountingHole_2.2mm_M2_ISO7380, F.Cu at (181.4, 173.7)
- added REF**: MountingHole_2.2mm_M2_ISO7380, MountingHole:MountingHole_2.2mm_M2_ISO7380, F.Cu at (224.6, 79.7)
- added REF**: MountingHole_2.2mm_M2_ISO7380, MountingHole:MountingHole_2.2mm_M2_ISO7380, F.Cu at (137.2, 79.4)
- added REF**: MountingHole_2.2mm_M2_ISO7380, MountingHole:MountingHole_2.2mm_M2_ISO7380, F.Cu at (243.5, 17.6)
- added REF**: MountingHole_2.2mm_M2_ISO7380, MountingHole:MountingHole_2.2mm_M2_ISO7380, F.Cu at (181.4, 111.5)
- added REF**: MountingHole_2.2mm_M2_ISO7380, MountingHole:MountingHole_2.2mm_M2_ISO7380, F.Cu at (65.8, 79.4)
- added REF**: MountingHole_2.2mm_M2_ISO7380, MountingHole:MountingHole_2.2mm_M2_ISO7380, F.Cu at (153.2, 173.7)
- added REF**: MountingHole_2.2mm_M2_ISO7380, MountingHole:MountingHole_2.2mm_M2_ISO7380, F.Cu at (64.8, 173.0)
- added REF**: MountingHole_2.2mm_M2_ISO7380, MountingHole:MountingHole_2.2mm_M2_ISO7380, F.Cu at (93.0, 173.0)
- added REF**: MountingHole_2.2mm_M2_ISO7380, MountingHole:MountingHole_2.2mm_M2_ISO7380, F.Cu at (272.6, 111.0)
- added REF**: MountingHole_2.2mm_M2_ISO7380, MountingHole:MountingHole_2.2mm_M2_ISO7380, F.Cu at (224.3, 173.3)
- added REF**: MountingHole_2.2mm_M2_ISO7380, MountingHole:MountingHole_2.2mm_M2_ISO7380, F.Cu at (272.6, 173.3)
- added REF**: MountingHole_2.2mm_M2_ISO7380, MountingHole:MountingHole_2.2mm_M2_ISO7380, F.Cu at (153.2, 79.9)
- added REF**: MountingHole_2.2mm_M2_ISO7380, MountingHole:MountingHole_2.2mm_M2_ISO7380, F.Cu at (196.2, 173.3)
- added REF**: MountingHole_2.2mm_M2_ISO7380, MountingHole:MountingHole_2.2mm_M2_ISO7380, F.Cu at (48.5, 110.5)
- added REF**: MountingHole_2.2mm_M2_ISO7380, MountingHole:MountingHole_2.2mm_M2_ISO7380, F.Cu at (243.5, 79.9)
- added REF**: MountingHole_2.2mm_M2_ISO7380, MountingHole:MountingHole_2.2mm_M2_ISO7380, F.Cu at (224.3, 111.0)
- added REF**: MountingHole_2.2mm_M2_ISO7380, MountingHole:MountingHole_2.2mm_M2_ISO7380, F.Cu at (224.5, 17.5)
- added REF**: MountingHole_2.2mm_M2_ISO7380, MountingHole:MountingHole_2.2mm_M2_ISO7380, F.Cu at (94.0, 17.1)
- added REF**: MountingHole_2.2mm_M2_ISO7380, MountingHole:MountingHole_2.2mm_M2_ISO7380, F.Cu at (196.4, 79.7)
- added REF**: MountingHole_2.2mm_M2_ISO7380, MountingHole:MountingHole_2.2mm_M2_ISO7380, F.Cu at (137.9, 110.6)
- added REF**: MountingHole_2.2mm_M2_ISO7380, MountingHole:MountingHole_2.2mm_M2_ISO7380, F.Cu at (109.7, 172.9)
- added REF**: MountingHole_2.2mm_M2_ISO7380, MountingHole:MountingHole_2.2mm_M2_ISO7380, F.Cu at (108.9, 17.1)
- added REF**: MountingHole_2.2mm_M2_ISO7380, MountingHole:MountingHole_2.2mm_M2_ISO7380, F.Cu at (153.1, 17.6)
- added REF**: MountingHole_2.2mm_M2_ISO7380, MountingHole:MountingHole_2.2mm_M2_ISO7380, F.Cu at (20.2, 110.4)
- added REF**: MountingHole_2.2mm_M2_ISO7380, MountingHole:MountingHole_2.2mm_M2_ISO7380, F.Cu at (153.1, 111.4)
- added REF**: MountingHole_2.2mm_M2_ISO7380, MountingHole:MountingHole_2.2mm_M2_ISO7380, F.Cu at (94.0, 79.4)
- added REF**: MountingHole_2.2mm_M2_ISO7380, MountingHole:MountingHole_2.2mm_M2_ISO7380, F.Cu at (271.7, 79.9)
- added REF**: MountingHole_2.2mm_M2_ISO7380, MountingHole:MountingHole_2.2mm_M2_ISO7380, F.Cu at (137.1, 17.1)
- added REF**: MountingHole_2.2mm_M2_ISO7380, MountingHole:MountingHole_2.2mm_M2_ISO7380, F.Cu at (20.3, 172.7)
- added REF**: MountingHole_2.2mm_M2_ISO7380, MountingHole:MountingHole_2.2mm_M2_ISO7380, F.Cu at (244.4, 173.3)
- added REF**: MountingHole_2.2mm_M2_ISO7380, MountingHole:MountingHole_2.2mm_M2_ISO7380, F.Cu at (137.9, 172.9)
- added REF**: MountingHole_2.2mm_M2_ISO7380, MountingHole:MountingHole_2.2mm_M2_ISO7380, F.Cu at (181.4, 79.9)
- added REF**: MountingHole_2.2mm_M2_ISO7380, MountingHole:MountingHole_2.2mm_M2_ISO7380, F.Cu at (244.4, 111.0)
- added REF**: MountingHole_2.2mm_M2_ISO7380, MountingHole:MountingHole_2.2mm_M2_ISO7380, F.Cu at (181.4, 17.6)
- added REF**: MountingHole_2.2mm_M2_ISO7380, MountingHole:MountingHole_2.2mm_M2_ISO7380, F.Cu at (109.0, 79.4)
- added REF**: MountingHole_2.2mm_M2_ISO7380, MountingHole:MountingHole_2.2mm_M2_ISO7380, F.Cu at (65.7, 17.1)
- added REF**: MountingHole_2.2mm_M2_ISO7380, MountingHole:MountingHole_2.2mm_M2_ISO7380, F.Cu at (109.7, 110.6)
- added REF**: MountingHole_2.2mm_M2_ISO7380, MountingHole:MountingHole_2.2mm_M2_ISO7380, F.Cu at (196.1, 111.0)
- added REF**: MountingHole_2.2mm_M2_ISO7380, MountingHole:MountingHole_2.2mm_M2_ISO7380, F.Cu at (196.3, 17.5)
- added REF**: MountingHole_2.2mm_M2_ISO7380, MountingHole:MountingHole_2.2mm_M2_ISO7380, F.Cu at (93.0, 110.7)
- added REF**: MountingHole_2.2mm_M2_ISO7380, MountingHole:MountingHole_2.2mm_M2_ISO7380, F.Cu at (64.8, 110.7)
- added REF**: MountingHole_2.2mm_M2_ISO7380, MountingHole:MountingHole_2.2mm_M2_ISO7380, F.Cu at (271.7, 17.6)
- added REF**: MountingHole_2.2mm_M2_ISO7380, MountingHole:MountingHole_2.2mm_M2_ISO7380, F.Cu at (48.5, 172.7)
- added S_OUT1: SIGNAL_OUT, TestPoint:TestPoint_Keystone_5015_Micro-Minature, B.Cu at (167.3, 18.6)
- added S_OUT1: SIGNAL_OUT, TestPoint:TestPoint_Keystone_5015_Micro-Minature, B.Cu at (258.6, 112.0)
- added S_OUT1: SIGNAL_OUT, TestPoint:TestPoint_Keystone_5015_Micro-Minature, B.Cu at (257.7, 18.6)
- added S_OUT1: SIGNAL_OUT, TestPoint:TestPoint_Keystone_5015_Micro-Minature, B.Cu at (167.3, 112.4)
- added S_OUT1: SIGNAL_OUT, TestPoint:TestPoint_Keystone_5015_Micro-Minature, B.Cu at (79.0, 111.7)
- added S_OUT1: SIGNAL_OUT, TestPoint:TestPoint_Keystone_5015_Micro-Minature, B.Cu at (123.1, 18.1)
- added S_OUT1: SIGNAL_OUT, TestPoint:TestPoint_Keystone_5015_Micro-Minature, B.Cu at (210.3, 112.0)
- added S_OUT1: SIGNAL_OUT, TestPoint:TestPoint_Keystone_5015_Micro-Minature, B.Cu at (34.4, 111.4)
- added S_OUT1: SIGNAL_OUT, TestPoint:TestPoint_Keystone_5015_Micro-Minature, B.Cu at (210.5, 18.4)
- added S_OUT1: SIGNAL_OUT, TestPoint:TestPoint_Keystone_5015_Micro-Minature, B.Cu at (79.9, 18.1)
- added S_OUT1: SIGNAL_OUT, TestPoint:TestPoint_Keystone_5015_Micro-Minature, B.Cu at (123.9, 111.6)
- added VCC1: TestPoint, TestPoint:TestPoint_Keystone_5015_Micro-Minature, B.Cu at (175.6, 18.6)
- added VCC1: TestPoint, TestPoint:TestPoint_Keystone_5015_Micro-Minature, B.Cu at (87.3, 111.7)
- added VCC1: TestPoint, TestPoint:TestPoint_Keystone_5015_Micro-Minature, B.Cu at (42.7, 111.4)
- added VCC1: TestPoint, TestPoint:TestPoint_Keystone_5015_Micro-Minature, B.Cu at (175.6, 112.4)
- added VCC1: TestPoint, TestPoint:TestPoint_Keystone_5015_Micro-Minature, B.Cu at (266.9, 112.0)
- added VCC1: TestPoint, TestPoint:TestPoint_Keystone_5015_Micro-Minature, B.Cu at (218.6, 112.0)
- added VCC1: TestPoint, TestPoint:TestPoint_Keystone_5015_Micro-Minature, B.Cu at (218.8, 18.4)
- added VCC1: TestPoint, TestPoint:TestPoint_Keystone_5015_Micro-Minature, B.Cu at (88.2, 18.1)
- added VCC1: TestPoint, TestPoint:TestPoint_Keystone_5015_Micro-Minature, B.Cu at (131.4, 18.1)
- added VCC1: TestPoint, TestPoint:TestPoint_Keystone_5015_Micro-Minature, B.Cu at (266.0, 18.6)
- added VCC1: TestPoint, TestPoint:TestPoint_Keystone_5015_Micro-Minature, B.Cu at (132.2, 111.6)
- moved R3 97.9 mm to (35.3, 22.8)
- moved R7 97.9 mm to (38.9, 22.9)
- moved REF** 97.9 mm to (48.2, 17.1)
- moved C2 97.9 mm to (35.2, 43.6)
- moved C3 97.9 mm to (31.6, 43.6)
- moved GND1 97.9 mm to (26.0, 18.1)
- moved R2 97.9 mm to (47.0, 43.8)
- moved R6 97.9 mm to (42.5, 22.9)
- moved RC4558IP2 97.9 mm to (23.9, 26.8)
- moved C1 97.9 mm to (40.1, 43.6)
- moved LM1458N1 97.9 mm to (27.7, 45.8)
- moved R1 97.9 mm to (44.0, 36.2)
- moved R4 97.9 mm to (31.8, 30.5)
- moved R5 97.9 mm to (46.2, 30.5)
- moved RC4558IP1 97.9 mm to (23.9, 39.8)
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Routing:
- net VCC: track 80.7 -> 968.4 mm
- net Net-(C1-Pad1): track 55.1 -> 717.5 mm
- net /PWD_1.65: track 44.8 -> 537.7 mm
- net /SIGNAL_2: track 44.1 -> 528.9 mm
- net Net-(R6-Pad1): track 41.8 -> 501.6 mm
- net /SIGNAL_1: track 38.8 -> 466.1 mm
- net Net-(C1-Pad2): track 30.3 -> 363.6 mm
- net Net-(R7-Pad1): track 16.7 -> 200.7 mm
- net Net-(R3-Pad2): track 16.7 -> 200.2 mm
- net Net-(C3-Pad1): track 10.1 -> 121.8 mm
- net unconnected-(LM1458N1-Pad6): track 0.14 -> 1.64 mm
Other:
- board size 33.3 x 62 mm -> 257.7 x 161.4 mm
